File: IO-Boards/GX700-PWB(F)/GX700-PWB/GX700-PWB.sch (KiCad schematic (older format))
At the start: 85 parts, among them CN33 Conn_01x10, CN34 Conn_01x10, CN35 Conn_01x10, U14 74LS273, U3 74LS273, U34 74LS273, U9 74LS175

Commit message: Added rough draft of Stage IO board
Connections:
- net EH? renamed ISOLATED-COMMON
Other:
- note added: "On DDR this is the Neon ouput"
- note added: "On DDR this is the P1 pad ouput"
- note added: "On DDR this is the P2 pad ouput"
- note added: "On DDR this is the cabinet lighting ouput"
Changed lines of the file:
@@
 Wire Wire Line
 	5050 7800 5850 7800
-Text GLabel 4300 8000 0    50   Input ~ 0
-EH?
 Wire Wire Line
 	4300 8000 4400 8000
@@
 Wire Wire Line
 	5050 4000 5850 4000
-Text GLabel 4300 4200 0    50   Input ~ 0
-EH?
 Wire Wire Line
 	4300 4200 4400 4200
@@
 	11200 4000 12000 4000
 Text GLabel 10450 4200 0    50   Input ~ 0
-EH?
+ISOLATED-COMMON
 Wire Wire Line
 	10450 4200 10550 4200
@@
 Wire Wire Line
 	10600 7100 10950 7100
-Text GLabel 10500 7100 0    50   Input ~ 0
-EH?
 Wire Wire Line
 	10500 7100 10600 7100
@@
 Text Notes 12400 8050 0    50   ~ 0
 OUTPUT 4
+Text GLabel 10500 7100 0    50   Input ~ 0
+ISOLATED-COMMON
+Text GLabel 4300 4200 0    50   Input ~ 0
+ISOLATED-COMMON
+Text GLabel 4300 8000 0    50   Input ~ 0
+ISOLATED-COMMON
+Text Notes 6900 7750 0    50   ~ 0
+On DDR this is the Neon ouput
+Text Notes 750  4050 0    50   ~ 0
+On DDR this is the P1 pad ouput
+Text Notes 750  7850 0    50   ~ 0
+On DDR this is the P2 pad ouput
+Text Notes 6950 4050 0    50   ~ 0
+On DDR this is the cabinet lighting ouput
 $EndSCHEMATC
