File: IO-Boards/GN845-PWB(B)/GN845-PWB/GN845-PWB.sch (KiCad schematic (older format))
At the start: 98 parts, among them CN1 B13PSHF1A, CN2 B11PSHF1A, CN3 B11PSHF1A, CN4 B11PSHF1A, CN5 B11PSHF1A, CN6 B11PSHF1A

Commit message: Added power input to GN845
Parts:
- added C1: 330uf 14v, Capacitor_THT:CP_Radial_D8.0mm_P3.50mm, symbol Device:CP1_Small
- added C23: 330uf 50v, Capacitor_THT:CP_Radial_D8.0mm_P3.50mm, symbol Device:CP1_Small
- added C24: 0.1uf 50v, Capacitor_THT:C_Disc_D4.7mm_W2.5mm_P5.00mm, symbol Device:C_Small
- added C3, C? (x2): 100n 25v, Capacitor_THT:C_Axial_L3.8mm_D2.6mm_P10.00mm_Horizontal, symbol Device:C_Small
- added C50, C? (x9): EMI_Filter_LCL, Connector_PinSocket_2.54mm:PinSocket_1x03_P2.54mm_Vertical, symbol Device:EMI_Filter_LCL
- added CN7: B4P-VH, Connector_JST:JST_VH_B4P-VH-B_1x04_P3.96mm_Vertical, symbol Connector_Generic:Conn_01x04
- added D1: 1N4001, Diode_THT:D_DO-41_SOD81_P10.16mm_Horizontal, symbol Diode:1N4001
- added U?: L7805, symbol Regulator_Linear:L7805
- C17, C4, C6, C7, C9: value 10n -> 100n
- gave numbers to parts that had none: 1
Connections:
- net labels added: LIGHT-GND
- wire segments 502 -> 593
Other:
- moved on the sheet: 10E, 7B?F, H?, JP?, JTAG

Commit message: Small updates
Connections:
- net at 10H.3, 10H?.3, 10H?.3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: now also C11.2, C12.2, C13.2, C14.2
- net 10E-10 renamed J-DN
- net 10E-11 renamed J-UP
- net 10E-7 renamed BT-C
- net 10E-8 renamed J-RT
- net 10E-9 renamed J-LF
- net J-LF: no longer 10H?.2
- new net J-LT: 10H?.2
Changed lines of the file:
@@
 	6800 3400 6800 2050
 Text GLabel 6300 2400 0    50   Input ~ 0
-10E-7
+BT-C
 Wire Wire Line
 	6300 2400 7500 2400
 Text GLabel 6300 2700 0    50   Input ~ 0
-10E-8
+J-RT
 Wire Wire Line
 	6300 2700 7500 2700
 Text GLabel 6300 3000 0    50   Input ~ 0
-10E-9
+J-LT
 Wire Wire Line
 	6300 3000 7500 3000
 Text GLabel 6300 3300 0    50   Input ~ 0
-10E-10
+J-DN
 Wire Wire Line
 	6300 3300 7500 3300
 Text GLabel 6300 3600 0    50   Input ~ 0
-10E-11
+J-UP
 Wire Wire Line
 	6300 3600 7500 3600
@@
 	7400 2450 9100 2450
 Wire Notes Line
-	9250 2800 10550 2800
-Wire Notes Line
 	10550 2800 10550 2500
 Wire Notes Line
@@
 	10850 4500 10850 7800
 Text GLabel 13250 7400 0    50   Input ~ 0
-10E-7
+BT-C
 Text GLabel 13250 7500 0    50   Input ~ 0
-10E-8
+J-RT
 Text GLabel 13250 7600 0    50   Input ~ 0
-10E-9
+J-LF
 Text GLabel 13250 7700 0    50   Input ~ 0
-10E-10
+J-DN
 Text GLabel 13250 7800 0    50   Input ~ 0
-10E-11
+J-UP
 Wire Wire Line
 	13350 7400 13250 7400
@@
 	9250 3800 9400 3800
 Wire Notes Line
-	9100 4150 9250 4150
-Wire Notes Line
-	9250 4150 9250 2800
-Wire Notes Line
 	9100 2450 9100 4150
 Wire Notes Line
@@
 	1    0    0    -1
 $EndComp
+Wire Wire Line
+	8550 3600 8700 3600
+Connection ~ 8550 3600
+Connection ~ 8700 3600
+Wire Wire Line
+	8700 3600 8850 3600
+Connection ~ 8850 3600
+Wire Wire Line
+	8850 3600 9000 3600
+Connection ~ 9000 3600
+Wire Wire Line
+	9000 3600 9150 3600
+Wire Notes Line
+	9200 2800 9200 4150
+Wire Notes Line
+	9200 2800 10550 2800
+Wire Notes Line
+	9200 4150 9100 4150
 $EndSCHEMATC
