File: Schematics/Ksys573.kicad_pcb (KiCad board)
At the start: 4 copper layers, 295 x 285 mm, 37 parts, among them CN1 B6P-VH, CN2 VGA-DSUB15, U1 27C040, U2 ADC0834

Commit message: Added GE675-PWB(A)
IO Board for Fisherman's Bait 3
Parts:
- added 10S1: 74LS245, Package_SO:SO-20_5.3x12.6mm_P1.27mm, F.Cu at (169.0, 284.0)
- added 10T1: ZBDS5101-8PT, Package_SO:SOIC-16_4.55x10.3mm_P1.27mm, F.Cu at (155.0, 278.0)
- added 12S1: 74LS245, Package_SO:SO-20_5.3x12.6mm_P1.27mm, F.Cu at (169.0, 266.0)
- added 12T1: ZBDS5101-8PT, Package_SO:SOIC-16_4.55x10.3mm_P1.27mm, F.Cu at (155.0, 265.0)
- added 13T1: ZBDS5101-8PT, Package_SO:SOIC-16_4.55x10.3mm_P1.27mm, F.Cu at (155.0, 252.0)
- added 14S1: 74LS245, Package_SO:SO-20_5.3x12.6mm_P1.27mm, F.Cu at (169.0, 251.0)
- added 21C1: 74LS74, Package_SO:SO-14_3.9x8.65mm_P1.27mm, F.Cu at (382.0, 199.0)
- added 22D1: 74LS273, Package_SO:SO-20_5.3x12.6mm_P1.27mm, F.Cu at (365.0, 197.0)
- added 22E1: 74LS273, Package_SO:SO-20_5.3x12.6mm_P1.27mm, F.Cu at (347.0, 197.0)
- added 24E1: 74LS14, Package_SO:SO-14_3.9x8.65mm_P1.27mm, F.Cu at (347.0, 180.0)
- added 35H1: 74LS125, Package_SO:SO-14_3.9x8.65mm_P1.27mm, F.Cu at (281.0, 91.0)
- added 3T1: EMI_Filter_LCL, Connector_PinSocket_2.54mm:PinSocket_1x03_P2.54mm_Vertical, F.Cu at (223.6, 238.1)
- added 4T1: EMI_Filter_LCL, Connector_PinSocket_2.54mm:PinSocket_1x03_P2.54mm_Vertical, F.Cu at (194.7, 250.0)
- added 5T1: EMI_Filter_LCL, Connector_PinSocket_2.54mm:PinSocket_1x03_P2.54mm_Vertical, F.Cu at (199.3, 250.0)
- added CN15: B4P-VH, Connector_JST:JST_VH_B4P-VH-B_1x04_P3.96mm_Vertical, F.Cu at (136.0, 338.0)
- added CN2I1: ATA-IDE, Connector_PinSocket_2.54mm:PinSocket_2x20_P2.54mm_Vertical, F.Cu at (143.5, 240.5)
- added RA4: 2.2k, Resistor_SMD:R_Array_Convex_5x1206, F.Cu at (312.3, 234.5)
- added U1: M48T58Y, Package_DIP:DIP-28_W15.24mm_Socket, F.Cu at (301.0, 203.0)
- added U3: 74LS74, Package_SO:SO-14_3.9x8.65mm_P1.27mm, F.Cu at (313.0, 130.0)
- added U4: KONAMI-058232, Arcade:KONAMI-SIP-14, F.Cu at (370.0, 313.0)
- added U71: 22J-X700A1 XC9536, Package_LCC:PLCC-44_SMD-Socket, F.Cu at (268.0, 187.0)
- moved 10B1 230.5 mm to (391.0, 295.0), turned to 180 degrees
- moved 12B1 213.8 mm to (391.0, 280.0), turned to 180 degrees
- moved 14B1 200.0 mm to (391.0, 264.0), turned to 180 degrees
- moved 15B1 197.4 mm to (391.0, 247.0), turned to 180 degrees
- moved U2 152.4 mm to (364.0, 180.0), turned to 180 degrees
- moved 20C1 123.6 mm to (348.3, 147.6)
- moved 36A1 123.6 mm to (353.1, 138.3)
- moved 15B2 123.6 mm to (343.4, 138.3)
- moved 25B1 122.5 mm to (338.0, 154.0)
- moved CN1 96.3 mm to (381.0, 101.0), turned to 270 degrees
- moved RA1 59.7 mm to (364.0, 267.0)
- moved EXT-IN-CN1 50.2 mm to (387.0, 222.0), turned to 90 degrees
- moved RA3 35.9 mm to (364.0, 239.0)
- moved ANALOG-CN1 26.5 mm to (372.0, 142.0), turned to 90 degrees
- moved 13E1 13.5 mm to (348.0, 259.0)
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- renumbered U1 to 22G1
Connections:
- net 35H-2 renamed EXO-CLK
- net Net-(13E1-Pad32) renamed CART-39
- net Net-(13E1-Pad33) renamed CART-38
- net Net-(13E1-Pad34) renamed CART-37
- net Net-(13E1-Pad35) renamed CART-36
- net Net-(13E1-Pad36) renamed CART-35
- net Net-(13E1-Pad37) renamed CART-34
- net Net-(13E1-Pad38) renamed CART-33
- net Net-(18E1-Pad36) renamed 18E-36
- net Net-(18E1-Pad37) renamed 18E-37
- net Net-(18E1-Pad38) renamed 18E-38
- net Net-(18E1-Pad50) renamed 18E-50
- net Net-(18E1-Pad51) renamed 18E-51
- net Net-(18E1-Pad52) renamed 18E-52
- 13E1 pad 39: Net-(13E1-Pad39) -> 18E-25
- 13E1 pad 40: GND -> 18E-26
- 13E1 pad 41: Net-(13E1-Pad41) -> GND
- 13E1 pad 45: +5V -> Net-(13E1-Pad45)
- 13E1 pad 46: Net-(13E1-Pad46) -> +5V
- 13E1 pad 48: 18E-17 -> Net-(13E1-Pad48)
- 13E1 pad 49: 18E-18 -> 18E-17
- 13E1 pad 50: GND -> 18E-18
- 13E1 pad 83: 058232-2 -> 058232-4
- 13E1 pad 84: 058232-3 -> 058232-5
- 13E1 pad 94: Net-(13E1-Pad94) -> JVS-S-IN
- 18E1 pad 1: Net-(18E1-Pad1) -> 22E-2
- 18E1 pad 11: Net-(18E1-Pad11) -> JVS-S-IN
- 18E1 pad 2: Net-(18E1-Pad2) -> 22E-5
- 18E1 pad 25: Net-(18E1-Pad25) -> 18E-25
- 18E1 pad 26: Net-(18E1-Pad26) -> 18E-26
- 18E1 pad 27: Net-(13E1-Pad41) -> Net-(13E1-Pad42)
- 18E1 pad 28: Net-(13E1-Pad42) -> Net-(13E1-Pad43)
- 18E1 pad 29: Net-(13E1-Pad43) -> Net-(13E1-Pad44)
- 18E1 pad 30: Net-(13E1-Pad44) -> Net-(13E1-Pad45)
- 18E1 pad 31: Net-(13E1-Pad46) -> Net-(13E1-Pad47)
- 18E1 pad 32: Net-(13E1-Pad47) -> Net-(13E1-Pad48)
- 18E1 pad 34: Net-(18E1-Pad34) -> 18E-34
- 18E1 pad 35: Net-(18E1-Pad35) -> 18E-35
- 18E1 pad 39: Net-(18E1-Pad39) -> 22D-2
- 18E1 pad 4: Net-(18E1-Pad4) -> GND
- 18E1 pad 40: Net-(18E1-Pad40) -> 22D-5
- 18E1 pad 41: Net-(18E1-Pad41) -> 22D-6
- 18E1 pad 42: Net-(18E1-Pad42) -> 22D-9
- 18E1 pad 43: Net-(18E1-Pad43) -> 22D-12
- 18E1 pad 44: Net-(18E1-Pad44) -> 22D-15
- 18E1 pad 45: Net-(18E1-Pad45) -> 22D-16
- 18E1 pad 46: Net-(18E1-Pad46) -> 22D-19
- 18E1 pad 53: Net-(18E1-Pad53) -> 21C-1
- 18E1 pad 54: Net-(18E1-Pad54) -> 21C-11
- 18E1 pad 59: Net-(18E1-Pad59) -> 22E-19
- 18E1 pad 60: Net-(18E1-Pad60) -> 22E-16
- 18E1 pad 61: Net-(18E1-Pad61) -> 22E-15
- 18E1 pad 62: Net-(18E1-Pad62) -> 22E-12
- 18E1 pad 63: Net-(18E1-Pad63) -> 22E-9
- 18E1 pad 64: Net-(18E1-Pad64) -> 22E-6
- 22G1 pad 22: Net-(U1-Pad22) -> GND
- 22G1 pad 24: Net-(U1-Pad24) -> PCPU-~BIOS
- 25B1 pad 15: 24E-9 -> JVS-SENSE
- JAMMA1 pad A25: Net-(2B1-Pad3) -> EXT-IN-7
- JAMMA1 pad B25: Net-(2B1-Pad3) -> EXT-IN-8

Commit message: Flash fixes, security cart done, most logic figured
Parts:
- added 12B2: ZBDS5101-8PT, Package_SO:SOIC-16_4.55x10.3mm_P1.27mm, F.Cu at (463.0, 199.1)
- added 13E2: KONAMI_056879, Package_QFP:TQFP-120_14x14mm_P0.4mm, F.Cu at (540.9, 141.4)
- added 22M1: 74LCX245, Package_SO:SSOP-20_4.4x6.5mm_P0.65mm, F.Cu at (557.0, 164.8)
- added 22N1: 74LCX245, Package_SO:SSOP-20_4.4x6.5mm_P0.65mm, F.Cu at (565.3, 164.8)
- added 22Q1: 74LCX245, Package_SO:SSOP-20_4.4x6.5mm_P0.65mm, F.Cu at (577.9, 162.9)
- added 23L1: 74F245, Package_SO:SO-20_5.3x12.6mm_P1.27mm, F.Cu at (565.5, 139.5)
- added 24E2: 74LS14, Package_SO:SO-14_3.9x8.65mm_P1.27mm, F.Cu at (585.1, 151.6)
- added 25R1: U102, Connector_PinHeader_2.54mm:PinHeader_1x03_P2.54mm_Vertical, F.Cu at (483.9, 195.5)
- added 25S1: U101, Connector_PinHeader_2.54mm:PinHeader_1x03_P2.54mm_Vertical, F.Cu at (479.3, 195.5)
- added 25T1: S240, Connector_PinHeader_2.54mm:PinHeader_2x04_P2.54mm_Vertical, F.Cu at (576.0, 148.9)
- added 26D1: ZBF503D-00, Resistor_THT:R_Axial_DIN0204_L3.6mm_D1.6mm_P5.08mm_Horizontal, F.Cu at (465.5, 216.8)
- added 27F1: 74LS273, Package_SO:SO-20_5.3x12.6mm_P1.27mm, F.Cu at (547.6, 157.4)
- added 27G1: 74LS273, Package_SO:SO-20_5.3x12.6mm_P1.27mm, F.Cu at (558.0, 153.6)
- added 27H1: 29F016-TSOP-SP, Package_SO:TSOP-I-48_18.4x12mm_P0.5mm, F.Cu at (481.5, 179.8)
- added 27J1: 29F016-TSOP-SP, Package_SO:TSOP-I-48_18.4x12mm_P0.5mm, F.Cu at (481.5, 166.3)
- added 27L1: 29F016-TSOP-SP, Package_SO:TSOP-I-48_18.4x12mm_P0.5mm, F.Cu at (476.0, 139.2)
- added 27M1: 29F016-TSOP-SP, Package_SO:TSOP-I-48_18.4x12mm_P0.5mm, F.Cu at (437.2, 181.5)
- added 27N1: 74F245, Package_SO:SO-20_5.3x12.6mm_P1.27mm, F.Cu at (586.4, 139.5)
- added 28E1: 74LS07, Package_SO:SO-14_5.3x10.2mm_P1.27mm, F.Cu at (441.8, 214.0)
- added 29D1: ZBF503D-00, Resistor_THT:R_Axial_DIN0204_L3.6mm_D1.6mm_P5.08mm_Horizontal, F.Cu at (448.5, 218.0)
- added 29E1: 74LS07, Package_SO:SO-14_5.3x10.2mm_P1.27mm, F.Cu at (431.3, 214.0)
- added 29G1: 74LS139, Package_SO:SOIC-16_4.55x10.3mm_P1.27mm, F.Cu at (514.0, 138.3)
- added 2C1: EVQ-PC1, Button_Switch_THT:SW_Tactile_SPST_Angled_PTS645Vx58-2LFS, F.Cu at (456.5, 211.5)
- added 30N1: 74F245, Package_SO:SO-20_5.3x12.6mm_P1.27mm, F.Cu at (568.5, 153.6)
- added 31H1: 29F016-TSOP-SP, Package_SO:TSOP-I-48_18.4x12mm_P0.5mm, F.Cu at (476.0, 152.7)
- added 31J1: 29F016-TSOP-SP, Package_SO:TSOP-I-48_18.4x12mm_P0.5mm, F.Cu at (459.3, 176.5)
- added 31L1: 29F016-TSOP-SP, Package_SO:TSOP-I-48_18.4x12mm_P0.5mm, F.Cu at (498.1, 139.2)
- added 31M1: 29F016-TSOP-SP, Package_SO:TSOP-I-48_18.4x12mm_P0.5mm, F.Cu at (498.1, 152.7)
- added 32N1: 74F245, Package_SO:SO-20_5.3x12.6mm_P1.27mm, F.Cu at (576.0, 139.5)
- added 35J1: 74LS125, Package_SO:SO-14_3.9x8.65mm_P1.27mm, F.Cu at (546.6, 178.8)
- added 35K1: 74LS273, Package_SO:SO-20_5.3x12.6mm_P1.27mm, F.Cu at (537.1, 180.7)
- added C209: 10n, Capacitor_SMD:C_0805_2012Metric, F.Cu at (538.6, 169.0)
- added C38: 10n, Capacitor_SMD:C_0805_2012Metric, F.Cu at (534.1, 166.0)
- added C39: 10n, Capacitor_SMD:C_0805_2012Metric, F.Cu at (538.6, 166.0)
- added C40: 10n, Capacitor_SMD:C_0805_2012Metric, F.Cu at (534.1, 169.0)
- added C41: 10n, Capacitor_SMD:C_0805_2012Metric, F.Cu at (543.0, 166.0)
- added C42: 10n, Capacitor_SMD:C_0805_2012Metric, F.Cu at (543.0, 169.0)
- added C43: 10n, Capacitor_SMD:C_0805_2012Metric, F.Cu at (544.6, 185.4)
- added CN5: B12PSHF1A, Connector_JST:JST_NH_B12P_SHD, F.Cu at (442.2, 200.8)
- added JP5: Jumper_NO_Small, Connector_PinSocket_2.54mm:PinSocket_1x02_P2.54mm_Vertical, F.Cu at (584.4, 159.1)
- added R288: 100, Resistor_SMD:R_0805_2012Metric, F.Cu at (547.5, 168.9)
- added R289: 470, Resistor_SMD:R_0805_2012Metric, F.Cu at (547.5, 166.0)
- added RA5: 4.7k, Resistor_SMD:R_Array_Convex_5x1206, F.Cu at (592.1, 152.3)
- added RA6: 4.7k, Resistor_SMD:R_Array_Convex_5x1206, F.Cu at (594.4, 144.3)
- added RA7: 4.7k, Resistor_SMD:R_Array_Convex_5x1206, F.Cu at (594.4, 136.4)
- added RA8: 4.7k, Resistor_SMD:R_Array_Convex_5x1206, F.Cu at (553.5, 177.6)
- added RA9: 4.7k, Resistor_SMD:R_Array_Convex_5x1206, F.Cu at (553.5, 185.6)
- U1: value M48T58Y -> KONAMI-058232; footprint Package_DIP:DIP-28_W15.24mm_Socket -> Arcade:KONAMI-SIP-14
- U4: value KONAMI-058232 -> M48T58Y; footprint Arcade:KONAMI-SIP-14 -> Package_DIP:DIP-28_W15.24mm_Socket
- moved 22E1 215.9 mm to (555.1, 139.5), turned to 0 degrees
- moved U4 194.6 mm to (447.6, 134.5), turned to 0 degrees
- moved 22D1 176.6 mm to (537.1, 157.4), turned to 0 degrees
- moved U1 138.8 mm to (439.8, 207.3), turned to 0 degrees
- moved 24E1 125.0 mm to (468.3, 210.2), turned to 0 degrees
- moved 22G1 124.7 mm to (428.2, 134.5), turned to 0 degrees
- moved 21C1 120.7 mm to (502.7, 198.3), turned to 0 degrees
Connections:
- net /IDE/PSX-DATA-0 renamed /IDE/IO-DATA-0
- net /IDE/PSX-DATA-1 renamed /IDE/IO-DATA-1
- net /IDE/PSX-DATA-10 renamed /IDE/IO-DATA-10
- net /IDE/PSX-DATA-11 renamed /IDE/IO-DATA-11
- net /IDE/PSX-DATA-12 renamed /IDE/IO-DATA-12
- net /IDE/PSX-DATA-13 renamed /IDE/IO-DATA-13
- net /IDE/PSX-DATA-14 renamed /IDE/IO-DATA-14
- net /IDE/PSX-DATA-15 renamed /IDE/IO-DATA-15
- net /IDE/PSX-DATA-2 renamed /IDE/IO-DATA-2
- net /IDE/PSX-DATA-3 renamed /IDE/IO-DATA-3
- net /IDE/PSX-DATA-4 renamed /IDE/IO-DATA-4
- net /IDE/PSX-DATA-5 renamed /IDE/IO-DATA-5
- net /IDE/PSX-DATA-6 renamed /IDE/IO-DATA-6
- net /IDE/PSX-DATA-7 renamed /IDE/IO-DATA-7
- net /IDE/PSX-DATA-8 renamed /IDE/IO-DATA-8
- net /IDE/PSX-DATA-9 renamed /IDE/IO-DATA-9
- net Net-(U71-Pad33) renamed U71-33
- net Net-(U71-Pad39) renamed U71-39
- net PSX-C-~RTS renamed PSX-~RTS
- net ~PSX-RST? renamed U17-3
- net ~PSX-WR renamed U17-2
- 13E1 pad 101: GND -> (no net)
- 13E1 pad 102: 13E-102 -> (no net)
- 13E1 pad 103: /IO-ADDR-1 -> (no net)
- 13E1 pad 104: /IO-ADDR-2 -> (no net)
- 13E1 pad 105: /IO-ADDR-3 -> (no net)
- 13E1 pad 106: +5V -> (no net)
- 13E1 pad 107: P1LFIN -> (no net)
- 13E1 pad 108: P1RTIN -> (no net)
- 13E1 pad 109: P1UPIN -> (no net)
- 13E1 pad 110: P1DNIN -> (no net)
- 13E1 pad 31: GND -> (no net)
- 13E1 pad 32: CART-39 -> (no net)
- 13E1 pad 33: CART-38 -> (no net)
- 13E1 pad 34: CART-37 -> (no net)
- 13E1 pad 35: CART-36 -> (no net)
- 13E1 pad 36: CART-35 -> (no net)
- 13E1 pad 37: CART-34 -> (no net)
- 13E1 pad 38: CART-33 -> (no net)
- 13E1 pad 39: 18E-25 -> (no net)
- 13E1 pad 40: 18E-26 -> (no net)
- 13E1 pad 90: ~IO-RST -> EXP-A10
- 13T1 pad 10: /IDE/IDE-CS0 -> /IDE/IDE-WRITE
- 13T1 pad 11: /IDE/IDE-A0 -> /IDE/IDE-READ
- 13T1 pad 12: /IDE/IDE-A2 -> /IDE/IDE-A1
- 13T1 pad 13: /IDE/IDE-A1 -> /IDE/IDE-A2
- 13T1 pad 14: /IDE/IDE-READ -> /IDE/IDE-A0
- 13T1 pad 15: /IDE/IDE-WRITE -> /IDE/IDE-CS0
- 13T1 pad 16: ~ATA-RST -> /IDE/IDE-CS1
- 13T1 pad 9: /IDE/IDE-CS1 -> ~ATA-RST
- 14S1 pad 1: IDE-AB -> +5V
- 14S1 pad 19: IDE-CE -> GND
- 14S1 pad 2: /IDE/PSX-AD- -> EXP-A10
- 14S1 pad 3: /IDE/PSX-AD- -> ~BUS-WR
- 14S1 pad 4: /IDE/PSX-AD- -> ~BUS-RD
- 14S1 pad 5: /IDE/PSX-AD- -> IO-ADDR-2
- 14S1 pad 6: /IDE/PSX-AD- -> IO-ADDR-3
- 14S1 pad 7: ~PSX-RD -> IO-ADDR-1
- 22D1 pad 1: LS273-~RST -> EXP-A10
- 22D1 pad 11: 22E-CP -> U17-39
- 22D1 pad 13: /PSX-DATA-12 -> /IO-DATA-12
- 22D1 pad 14: /PSX-DATA-13 -> /IO-DATA-13
- 22D1 pad 17: /PSX-DATA-14 -> /IO-DATA-14
- 22D1 pad 18: /PSX-DATA-15 -> /IO-DATA-15
- 22D1 pad 3: /PSX-DATA-8 -> /IO-DATA-8
- 22D1 pad 4: /PSX-DATA-9 -> /IO-DATA-9
- 22D1 pad 7: /PSX-DATA-10 -> /IO-DATA-10
- 22D1 pad 8: /PSX-DATA-11 -> /IO-DATA-11
- 22E1 pad 1: LS273-~RST -> EXP-A10
- 22E1 pad 11: 22E-CP -> U17-39
- 22E1 pad 13: /PSX-DATA-4 -> /IO-DATA-4
- 22E1 pad 14: /PSX-DATA-5 -> /IO-DATA-5
- 22E1 pad 17: /PSX-DATA-6 -> /IO-DATA-6
- 22E1 pad 18: /PSX-DATA-7 -> /IO-DATA-7
- 22E1 pad 3: /PSX-DATA-0 -> /IO-DATA-0
- 22E1 pad 4: /PSX-DATA-1 -> /IO-DATA-1
- 22E1 pad 7: /PSX-DATA-2 -> /IO-DATA-2
- 22E1 pad 8: /PSX-DATA-3 -> /IO-DATA-3
- 22G1 pad 10: /IO-ADDR-2 -> /ROM/IO-ADDR-2
- 22G1 pad 11: /IO-ADDR-1 -> /ROM/IO-ADDR-1
- 22G1 pad 12: /IO-ADDR-0 -> /ROM/IO-ADDR-0
- 22G1 pad 13: /IO-DATA-0 -> /ROM/IO-DATA-0
- 22G1 pad 14: /IO-DATA-1 -> /ROM/IO-DATA-1
- 22G1 pad 15: /IO-DATA-2 -> /ROM/IO-DATA-2
- 22G1 pad 17: /IO-DATA-3 -> /ROM/IO-DATA-3
- 22G1 pad 18: /IO-DATA-4 -> /ROM/IO-DATA-4
- 22G1 pad 19: /IO-DATA-5 -> /ROM/IO-DATA-5
- 22G1 pad 2: /IO-ADDR-16 -> /ROM/IO-ADDR-16
- 22G1 pad 20: /IO-DATA-6 -> /ROM/IO-DATA-6
- 22G1 pad 21: /IO-DATA-7 -> /ROM/IO-DATA-7
- 22G1 pad 23: /IO-ADDR-10 -> /ROM/IO-ADDR-10
- 22G1 pad 25: /IO-ADDR-11 -> /ROM/IO-ADDR-11
- 22G1 pad 26: /IO-ADDR-9 -> /ROM/IO-ADDR-9
- 22G1 pad 27: /IO-ADDR-8 -> /ROM/IO-ADDR-8
- 22G1 pad 28: /IO-ADDR-13 -> /ROM/IO-ADDR-13
- 22G1 pad 29: /IO-ADDR-14 -> /ROM/IO-ADDR-14
- 22G1 pad 3: /IO-ADDR-15 -> /ROM/IO-ADDR-15
- 22G1 pad 30: /IO-ADDR-17 -> /ROM/IO-ADDR-17
- 22G1 pad 31: /IO-ADDR-18 -> /ROM/IO-ADDR-18
- 22G1 pad 4: /IO-ADDR-12 -> /ROM/IO-ADDR-12
- 22G1 pad 5: /IO-ADDR-7 -> /ROM/IO-ADDR-7
- 22G1 pad 6: /IO-ADDR-6 -> /ROM/IO-ADDR-6
- 22G1 pad 7: /IO-ADDR-5 -> /ROM/IO-ADDR-5
- 22G1 pad 8: /IO-ADDR-4 -> /ROM/IO-ADDR-4
- 22G1 pad 9: /IO-ADDR-3 -> /ROM/IO-ADDR-3
- 24E1 pad 12: 35H-10 -> (no net)
- 24E1 pad 13: Net-(24E1-Pad13) -> (no net)
- 35H1 pad 10: 35H-10 -> Net-(24E2-Pad12)
- 35H1 pad 14: Net-(35H1-Pad14) -> (no net)
- 35H1 pad 5: Net-(13E1-Pad97) -> PSX-TX1
- 35H1 pad 6: CART-5 -> TX1
- 35H1 pad 7: GND -> (no net)
- CN2I1 pad 37: /IDE/IDE-CS1 -> /IDE/IDE-CS0
- CN2I1 pad 38: /IDE/IDE-CS0 -> /IDE/IDE-CS1
- U1 pad 1: Net-(U1-Pad1) -> +12V
- U1 pad 11: /IO-DATA-0 -> Net-(U1-Pad11)
- U1 pad 12: /IO-DATA-1 -> Net-(2C1-Pad1)
- U1 pad 13: /IO-DATA-2 -> EXP-A10
- U1 pad 14: GND -> (no net)
- U1 pad 2: Net-(U1-Pad2) -> COIN-CNT2
- U1 pad 3: Net-(U1-Pad3) -> COIN-CNT1
- U1 pad 4: Net-(U1-Pad4) -> 058232-4
- U1 pad 5: Net-(U1-Pad5) -> 058232-5
- U1 pad 6: Net-(U1-Pad6) -> GND
- U1 pad 7: Net-(U1-Pad7) -> GND
- U1 pad 8: Net-(U1-Pad8) -> +5V
- U1 pad 9: Net-(U1-Pad9) -> U71-43
- U4 pad 1: +12V -> Net-(U4-Pad1)
- U4 pad 11: Net-(U4-Pad11) -> /ROM/IO-DATA-0
- U4 pad 12: Net-(U4-Pad12) -> /ROM/IO-DATA-1
- U4 pad 13: (no net) -> /ROM/IO-DATA-2
- U4 pad 14: (no net) -> GND
- U4 pad 2: COIN-CNT2 -> Net-(U4-Pad2)
- U4 pad 3: COIN-CNT1 -> Net-(U4-Pad3)
- U4 pad 4: 058232-4 -> Net-(U4-Pad4)
- U4 pad 5: 058232-5 -> Net-(U4-Pad5)
- U4 pad 6: GND -> Net-(U4-Pad6)
- U4 pad 7: GND -> Net-(U4-Pad7)
- U4 pad 8: +5V -> Net-(U4-Pad8)
- U4 pad 9: 35J-11 -> Net-(U4-Pad9)
- U71 pad 4: Net-(U71-Pad4) -> U17-4
- U71 pad 43: 35J-11 -> U71-43
- U71 pad 7: Net-(U71-Pad7) -> U17-7
- U71 pad 8: Net-(U71-Pad8) -> IO-ADDR-23
- U71 pad 9: Net-(U71-Pad9) -> IO-ADDR-22
