File: Schematics/573-ROM.sch (KiCad schematic (older format))
At the start: 11 parts

Commit message: Flash fixes, security cart done, most logic figured
Parts:
- removed 13E?: KONAMI_056879, Package_QFP:TQFP-120_14x14mm_P0.4mm, symbol Arcade:KONAMI_056879
- added 29G1: 74LS139, Package_SO:SOIC-16_4.55x10.3mm_P1.27mm, symbol 74xx:74LS139
- gave numbers to parts that had none: 2
- renumbered 27H to 27H1, 27J to 27J1, 27L to 27L1, 27M to 27M1, 31H to 31H1, 31J to 31J1, 31L to 31L1, 31M to 31M1
Connections:
- net NVRAM-~WR: no longer 27H1.44 (~WE), 27J1.44 (~WE), 27L1.44 (~WE), 27M1.44 (~WE), 31H1.44 (~WE), 31J1.44 (~WE), 31L1.44 (~WE), 31M1.44 (~WE)
- net FLASH-CE0: now reaches 31H1.11 (~CE)
- net FLASH-CE0: now also 27H1.11 (~CE), 29G1.9 (O3)
- net ~RESET: now reaches 31H1.14 (~RESET)
- net ~RESET: now also 27H1.14 (~RESET), 27J1.14 (~RESET), 27L1.14 (~RESET), 27M1.14 (~RESET), 31J1.14 (~RESET), 31L1.14 (~RESET), 31M1.14 (~RESET)
- net ~BUS-RD: now reaches 31H1.43 (~OE)
- net ~BUS-RD: now also 27H1.43 (~OE), 27J1.43 (~OE), 27L1.43 (~OE), 27M1.43 (~OE), 31J1.43 (~OE), 31L1.43 (~OE), 31M1.43 (~OE)
- net FLASH-CE1: now reaches 31J1.11 (~CE)
- net FLASH-CE1: now also 27J1.11 (~CE), 29G1.10 (O2)
- net FLASH-CE2: now reaches 31L1.11 (~CE)
- net FLASH-CE2: now also 29G1.11 (O1)
- net FLASH-CE3: now reaches 31M1.11 (~CE)
- net FLASH-CE3: now also 27M1.11 (~CE), 29G1.12 (O0)
- net FLASH-C2: now reaches 27L1.11 (~CE)
- new net: 29G1.15 (E), 29G1.4 (O0)
- new net 27G-12: 29G1.2 (A0)
- new net 27G-15: 29G1.3 (A1)
- new net 27G-2: 29G1.14 (A0)
- new net 27G-5: 29G1.13 (A1)
- new net 29G-5: 29G1.5 (O1)
- new net 29G-6: 29G1.6 (O2)
- new net BUS-~WR: 27H1.44 (~WE), 27J1.44 (~WE), 27L1.44 (~WE), 27M1.44 (~WE), 31H1.44 (~WE), 31J1.44 (~WE), 31L1.44 (~WE), 31M1.44 (~WE)
- new net U17-37: 29G1.1 (E)
- no-connect marks 0 -> 1
Other:
- note added: "PCCARD 1 (T) CE"
- note added: "PCCARD 2 (B) CE"
- note removed: "Details in JAMMA.sch"

Commit message: 573 specific mostly mapped
Connections:
- net NVRAM-~WR is gone; now on net BUS-~WR: U4.27 (~WR)
- net RTC-FT: now reaches U4.1 (FT)
- net U71-40: now reaches U4.20 (~E1)
- net BUS-~RD: now reaches U4.22 (~OE)
- net PCPU-~BIOS renamed U71-19
Other:
- note added: "FLASH-4 U71-13"
- note added: "Flash starts at A1"
- note added: "Goes to KCUS 28"
Changed lines of the file:
@@
 Wire Wire Line
 	5850 10450 5950 10450
-Text GLabel 5550 10550 0    50   Input ~ 0
-PCPU-~BIOS
-Wire Wire Line
-	5550 10550 5950 10550
 Text Label 7400 9200 0    50   ~ 0
 IO-DATA
@@
 Wire Wire Line
 	9000 10350 9000 10450
-Wire Wire Line
-	8950 10100 9100 10100
-Text GLabel 8950 10100 0    50   Input ~ 0
-NVRAM-~WR
+Text GLabel 8950 10200 0    50   Input ~ 0
+BUS-~WR
 Text Label 8500 8350 0    50   ~ 0
 IO-ADDR-0
@@
 Wire Wire Line
 	13450 2650 13350 2650
+Text GLabel 5750 10550 0    50   Input ~ 0
+U71-19
+Wire Wire Line
+	5750 10550 5950 10550
+Text Notes 1900 7300 0    50   ~ 0
+FLASH-4 U71-13
+Text Notes 1900 7400 0    50   ~ 0
+Flash starts at A1
+Text GLabel 8950 9750 0    50   Input ~ 0
+U71-40
+Wire Wire Line
+	8950 9750 9100 9750
+Wire Wire Line
+	8950 10200 9100 10200
+Wire Wire Line
+	9100 10200 9100 10100
+Text GLabel 8950 10000 0    50   Input ~ 0
+BUS-~RD
+Wire Wire Line
+	8950 10000 9100 10000
+Text GLabel 10050 10350 2    50   Input ~ 0
+RTC-FT
+Wire Wire Line
+	10050 10350 9900 10350
 Wire Bus Line
 	14000 1400 14000 4150
@@
 Wire Bus Line
 	5300 8250 5300 10250
+Text Notes 10400 10400 0    50   ~ 0
+Goes to KCUS 28
 $EndSCHEMATC
