File: Schematics/Ksys573.sch (KiCad schematic (older format))
At the start: 37 parts, among them U71 22J-X700A1 XC9536

Commit message: Added GE675-PWB(A)
IO Board for Fisherman's Bait 3
Parts:
- added U1: M48T58Y, Package_DIP:DIP-28_W15.24mm_Socket, symbol RTC_ST:M48T58Y
- added U5: 29F016-TSOP-SP, symbol Memory_Flash:29F016-TSOP-SP
- gave numbers to parts that had none: 5
- renumbered 21C to 21C1, 22D to 22D1, 22E to 22E1, 22G to 22G1, 24E to 24E1, 27G to 27G1, 35H to 35H1
Connections:
- net labels added: NVRAM-~WR
- wire segments 207 -> 248
Other:
- moved on the sheet: 13E1G, 13E1H, 13E1K, 21C1A, 22D1, 22D2, 22E1, 22G1, 24E1F, 27G1, 35H1E, C265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

Commit message: Updated Schematics
PCMCIA is pinned out
Parts:
- removed unit 11 of 13E1
- removed 21C1: 74LS74, Package_SO:SO-14_3.9x8.65mm_P1.27mm, symbol 74xx:74LS74
- removed 22D1, 22E1: 74LS273, Package_SO:SO-20_5.3x12.6mm_P1.27mm, symbol 74xx:74LS273
- removed 22G1: 27C040, Package_DIP:DIP-32_W15.24mm_Socket, symbol Memory_EPROM:27C040
- removed 24E1: 74LS14, Package_SO:SO-14_3.9x8.65mm_P1.27mm, symbol 74xx:74LS14
- removed 27G1: 74LS273, symbol 74xx:74LS273
- removed unit 5 of 35H1
- removed C265, C274: 10n, symbol Device:C_Small
- removed U1: M48T58Y, Package_DIP:DIP-28_W15.24mm_Socket, symbol RTC_ST:M48T58Y
- removed U4: KONAMI-058232, Arcade:KONAMI-SIP-14, symbol Arcade:KONAMI-058232
- removed U5: 29F016-TSOP-SP, symbol Memory_Flash:29F016-TSOP-SP
- added 22N?, 22Q?: 74LCX245, Package_SO:SSOP-20_4.4x6.5mm_P0.65mm, symbol 74xx:74LS245
- added 23L?, 27N?, 30N?, 32N?: 74F245, Package_SO:SO-20_5.3x12.6mm_P1.27mm, symbol 74xx:74LS245
- added 24E?: 74LS14, Package_SO:SO-14_3.9x8.65mm_P1.27mm, symbol 74xx:74LS14
- added 27G?: 74LS273, Package_SO:SO-20_5.3x12.6mm_P1.27mm, symbol 74xx:74LS273
- added 29G?: 74LS139, Package_SO:SOIC-16_4.55x10.3mm_P1.27mm, symbol 74xx:74LS139
- added 29G?: 74LS139, symbol 74xx:74LS139
- added C? (x4): 10n, Capacitor_SMD:C_0805_2012Metric, symbol Device:C_Small
- added RA? (x6): 4.7k, Resistor_SMD:R_Array_Convex_5x1206, symbol Device:R_Dual_Network08_Split
Connections:
- net labels added: 22G-2, 22G-5, 22G-6, 27G-12, 27G-15, 27G-2, 27G-5, 29G-5, 29G-6, IO-ADDR-19, IO-ADDR-20, IO-ADDR-21, IO-ADDR-22, IO-ADDR-23, IO-DIR, IO-~CE, PSX-ADDR-0, PSX-ADDR-1, PSX-ADDR-10, PSX-ADDR-11, PSX-ADDR-12, PSX-ADDR-13, PSX-ADDR-14, PSX-ADDR-15, PSX-ADDR-16, PSX-ADDR-17, PSX-ADDR-18, PSX-ADDR-19, PSX-ADDR-2, PSX-ADDR-20, PSX-ADDR-21, PSX-ADDR-22, PSX-ADDR-23, PSX-ADDR-3, PSX-ADDR-4, PSX-ADDR-5, PSX-ADDR-6, PSX-ADDR-7, PSX-ADDR-8, PSX-ADDR-9, U17-37, U71-33, ~BUS-RD, ~BUS-WR, ~BUS-WR2, ~EXP-CE, ~PSX-EXP, ~PSX-RD, ~PSX-WR, ~PSX-WR2
- net labels removed: +12V, 058232-4, 058232-5, 13E-102, 18E-34, 21C-1, 22D-12, 22D-15, 22D-16, 22D-19, 22D-2, 22D-5, 22D-6, 22D-9, 22E-12, 22E-15, 22E-16, 22E-19, 22E-2, 22E-5, 22E-6, 22E-9, 22E-CP, COIN-CNT1, COIN-CNT2, IO-ADDR, P1DNIN, P1LFIN, P1RTIN, P1UPIN
- wire segments 248 -> 275
Other:
- note added: "3.3v to 5V for\nbus signals"
- note added: "PCCARD 1 (T) CE"
- note added: "PCCARD 2 (B) CE"
- note added: "Slot-0 PCMCIA CE Stuff"
- note removed: "Details in JAMMA.sch"
- note removed: "H8/6433\nPort B/AN"
- moved on the sheet: 22D2, C38, RA4A

Commit message: Fixed bugs
IDE Retrace, PCMCIA checked
Parts:
- removed 22D2: 74LS273, symbol 74xx:74LS273
- removed C38: 10n, symbol Device:C_Small
- added 22D?, 22E?: 74LS273, Package_SO:SO-20_5.3x12.6mm_P1.27mm, symbol 74xx:74LS273
- added 22M: 74LCX245, Package_SO:SSOP-20_4.4x6.5mm_P0.65mm, symbol 74xx:74LS245
- added 25T: S240, Connector_PinHeader_2.54mm:PinHeader_2x04_P2.54mm_Vertical, symbol Connector_Generic:Conn_02x04_Counter_Clockwise
- added C? (x2): 10n, Capacitor_SMD:C_0805_2012Metric, symbol Device:C_Small
Connections:
- net +5V: now also 22D?.20 (VCC), 22E?.20 (VCC), 22M.20 (VCC), C?.1, C?.1
- net GND: now also 22D?.10 (GND), 22E?.10 (GND), 22M.1 (A->B), 22M.10 (GND), 22M.19 (CE), C?.2, C?.2
- net IO-DATA-0: now also 22E?.3 (D0)
- net IO-DATA-1: now also 22E?.4 (D1)
- net IO-DATA-10: now also 22D?.7 (D2)
- net IO-DATA-11: now also 22D?.8 (D3)
- net IO-DATA-12: now also 22D?.13 (D4)
- net IO-DATA-13: now also 22D?.14 (D5)
- net IO-DATA-14: now also 22D?.17 (D6)
- net IO-DATA-15: now also 22D?.18 (D7)
- net IO-DATA-2: now also 22E?.7 (D2)
- net IO-DATA-3: now also 22E?.8 (D3)
- net IO-DATA-4: now also 22E?.13 (D4)
- net IO-DATA-5: now also 22E?.14 (D5)
- net IO-DATA-6: now also 22E?.17 (D6)
- net IO-DATA-7: now also 22E?.18 (D7)
- net IO-DATA-8: now also 22D?.3 (D0)
- net IO-DATA-9: now also 22D?.4 (D1)
- net LS273-~RST: now also 22D?.1 (~Mr), 22E?.1 (~Mr)
- net EXP-B14: now reaches 23L?.15 (B3)
- net ~PSX-DMACK5: now reaches 23L?.5 (A3)
- new net 22D-12: 22D?.12 (Q4)
- new net 22D-15: 22D?.15 (Q5)
- new net 22D-16: 22D?.16 (Q6)
- new net 22D-19: 22D?.19 (Q7)
- new net 22D-2: 22D?.2 (Q0)
- new net 22D-5: 22D?.5 (Q1)
- new net 22D-6: 22D?.6 (Q2)
- new net 22D-9: 22D?.9 (Q3)
- new net 22E-12: 22E?.12 (Q4)
- new net 22E-15: 22E?.15 (Q5)
- new net 22E-16: 22E?.16 (Q6)
- new net 22E-19: 22E?.19 (Q7)
- new net 22E-2: 22E?.2 (Q0)
- new net 22E-5: 22E?.5 (Q1)
- new net 22E-6: 22E?.6 (Q2)
- new net 22E-9: 22E?.9 (Q3)
- new net 22E-CP: 22D?.11 (Cp), 22E?.11 (Cp)
- new net 22M-13: 22M.13 (B5), 25T.4 (Pin_4), 25T.5 (Pin_5)
- new net 25T-6: 25T.3 (Pin_3), 25T.6 (Pin_6)
- new net 25T-7: 25T.2 (Pin_2), 25T.7 (Pin_7)
- new net 25T-8: 25T.1 (Pin_1), 25T.8 (Pin_8)
- new net PSX-~IRQ10: 22M.7 (A5)
Other:
- note added: "<— Direction"
- note added: "H8/6433\nPort B/AN"
- note added: "Yes this header is joined like this.\nNo, I do not know why."
- moved on the sheet: 22N?, 23L?, 24E?F, 29G?A, 29G?B, 30N?, 32N?, C?, H1, H10, H11, H12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

Commit message: Flash fixes, security cart done, most logic figured
Parts:
- removed 24E?: 74LS14, Package_SO:SO-14_3.9x8.65mm_P1.27mm, symbol 74xx:74LS14
- removed 29G?: 74LS139, Package_SO:SOIC-16_4.55x10.3mm_P1.27mm, symbol 74xx:74LS139
- removed 29G?: 74LS139, symbol 74xx:74LS139
- removed 35H1: 74LS125, Package_SO:SO-14_3.9x8.65mm_P1.27mm, symbol 74xx:74LS125
- removed U3: 74LS74, Package_SO:SO-14_3.9x8.65mm_P1.27mm, symbol 74xx:74LS74
- added 13E2: KONAMI_056879, Package_QFP:TQFP-120_14x14mm_P0.4mm, symbol Arcade:KONAMI_056879
- added 27F1: 74LS273, Package_SO:SO-20_5.3x12.6mm_P1.27mm, symbol 74xx:74LS273
- added CN21: TX15-30P-ST, symbol Connector_Generic:Conn_02x15_Row_Letter_First
- added JP5: Jumper_NO_Small, Connector_PinSocket_2.54mm:PinSocket_1x02_P2.54mm_Vertical, symbol Device:Jumper_NO_Small
- added R288: 100, Resistor_SMD:R_0805_2012Metric, symbol Device:R_Small
- added R289: 470, Resistor_SMD:R_0805_2012Metric, symbol Device:R_Small
- gave numbers to parts that had none: 18
- renumbered 22M to 22M1, 25T to 25T1
Connections:
- net 22G-2 is gone; now on net 27G-2: 27G1.2 (Q0)
- net 22G-5 is gone; now on net 27G-5: 27G1.5 (Q1)
- net IO-DIR is gone; now on net ~PSX-RD: 22N1.1 (A->B), 22Q1.1 (A->B)
- net +5V: now also 13E2.106, 27F1.20 (VCC), R289.1
- net 27G-12: now also 27G1.12 (Q4)
- net 27G-15: now also 27G1.15 (Q5)
- net GND: now also 22M1.17 (B1), 22M1.18 (B0), 13E2.101, 27F1.10 (GND), CN21.a10 (Pin_a10), CN21.a11 (Pin_a11), CN21.a12 (Pin_a12), CN21.a13 (Pin_a13), CN21.a14 (Pin_a14), CN21.a15 (Pin_a15), CN21.a5 (Pin_a5), CN21.a6 (Pin_a6), CN21.a7 (Pin_a7), CN21.a8 (Pin_a8), CN21.a9 (Pin_a9), CN21.b7 (Pin_b7), CN21.b9 (Pin_b9)
- net IO-ADDR-1: now also 13E2.103
- net IO-ADDR-2: now also 13E2.104
- net IO-ADDR-3: now also 13E2.105
- net IO-DATA-0: now also 27F1.3 (D0)
- net IO-DATA-1: now also 27F1.4 (D1)
- net IO-DATA-2: now also 27F1.7 (D2)
- net IO-DATA-3: now also 27F1.8 (D3)
- net IO-DATA-4: now also 27F1.13 (D4)
- net IO-DATA-5: now also 27F1.14 (D5)
- net IO-DATA-6: now also 27F1.17 (D6)
- net IO-DATA-7: now also 27F1.18 (D7)
- net LS273-~RST: now also 27F1.1 (~Mr); no longer 22D1.1 (~Mr), 22E1.1 (~Mr)
- net PSX-ADDR-10: now also CN21.a2 (Pin_a2)
- net PSX-ADDR-11: now also CN21.b2 (Pin_b2)
- net PSX-ADDR-16: now also CN21.a3 (Pin_a3)
- net PSX-ADDR-17: now also CN21.b3 (Pin_b3)
- net PSX-ADDR-18: now also CN21.a4 (Pin_a4)
- net PSX-ADDR-19: now also CN21.b4 (Pin_b4)
- net PSX-ADDR-8: now also CN21.a1 (Pin_a1)
- net PSX-ADDR-9: now also CN21.b1 (Pin_b1)
- net CART-28: now reaches 13E1.93
- net KCUS-98: now reaches 13E1.98
- net U71-39: now reaches U71.39 (I/O/GSR)
- net U17-4: now reaches U71.4 (M4)
- net U17-4: now also 27G1.11 (Cp)
- net U17-6: now reaches U71.6 (I/O/GCK2)
- net U17-7: now reaches U71.7 (I/O/GCK3)
- net U17-7: now also 27G1.19 (Q7)
- net 24E-13: now reaches 27G1.16 (Q6)
- net 27G-9: now reaches 27G1.9 (Q3)
- net at 23L1.16 (B2): now also R288.1, R289.2
- net CN21-B6: now reaches 23L1.17 (B1)
- net CN21-B6: now also CN21.b6 (Pin_b6), JP5.1
- net CN21-B5: now reaches 23L1.18 (B0)
- net CN21-B5: now also CN21.b5 (Pin_b5)
- net EXP-A10: now reaches 22M1.11 (B7)
- net EXP-A10: now also 22D1.1 (~Mr), 22E1.1 (~Mr)
- net DREQ5: now reaches 22M1.12 (B6)
- net RX1: now reaches 22M1.14 (B4)
- net ~DSR: now reaches 22M1.15 (B3)
- net ~CTS: now reaches 22M1.16 (B2)
- net PSX-~CTS: now reaches 22M1.4 (A2)
- net PSX-~DSR: now reaches 22M1.5 (A3)
- net PSX-RX: now reaches 22M1.6 (A4)
- net PSX-DREQ5: now reaches 22M1.8 (A6)
- net PSX-~RST: now reaches 22M1.9 (A7)
- net 22E-CP renamed U17-39
- net 22G-6 renamed 27G-6
- net IO-~CE renamed U17-35
- new net 13E-102: 13E2.102
- new net EXT-OUTPUT-0: 27F1.2 (Q0)
- new net EXT-OUTPUT-1: 27F1.5 (Q1)
- new net EXT-OUTPUT-2: 27F1.6 (Q2)
- new net EXT-OUTPUT-3: 27F1.9 (Q3)
- new net EXT-OUTPUT-4: 27F1.12 (Q4)
- new net EXT-OUTPUT-5: 27F1.15 (Q5)
- new net EXT-OUTPUT-6: 27F1.16 (Q6)
- new net EXT-OUTPUT-7: 27F1.19 (Q7)
- new net P1DNIN: 13E2.110
- new net P1LFIN: 13E2.107
- new net P1RTIN: 13E2.108
- new net P1UPIN: 13E2.109
- new net PSX-DOTCLK: CN21.b8 (Pin_b8)
- new net PSX-JOYCLK: CN21.b15 (Pin_b15)
- new net PSX-JOYCMD: CN21.b14 (Pin_b14)
- new net PSX-JOYDATA: CN21.b13 (Pin_b13)
- new net PSX-~IRQ7: CN21.b10 (Pin_b10)
- new net PSX-~JOY1: CN21.b12 (Pin_b12)
- new net PSX-~JOY2: CN21.b11 (Pin_b11)
- new net U17-43: 27F1.11 (Cp)
- new net VGA-14: JP5.2
- new net VGA-CSYNC: R288.2
- no-connect marks 2 -> 3
Other:
- note added: "27F CP"
- note added: "27G CP\n"
- note added: "27G-19 OUT 8"
- note added: "29G Low"
- note added: "Details in JAMMA.sch"
- note added: "Direction —>"
- note added: "External Outputs Header\nIn JAMMA-IO"
- note added: "Goes under CPU"
- note added: "H8 16-bit data port"
- note added: "PCMCIA A22-A25"
- note added: "These two stop here?"
- note removed: "PCCARD 1 (T) CE"
- note removed: "PCCARD 2 (B) CE"
- moved on the sheet: 22D1, 22E1, 22M1, 23L1, 25T1, 27G1, 27N1, 30N1, 32N1, C209, C38, C39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

Commit message: 573 specific mostly mapped
Parts:
- added 26E: 74LS74, Package_SO:SO-14_5.3x10.2mm_P1.27mm, symbol 74xx:74LS74
- added CN10: TX15-80P-ST, symbol Connector_Generic:Conn_02x40_Row_Letter_First
Connections:
- net 13E-102 is gone; now on net U71-26: 13E2.102
- net +5V: now also 13E1.99, U71.20 (M15), 26E.10 (~S), 26E.4 (~S); no longer 22M1.20 (VCC), 22N1.20 (VCC), 22Q1.20 (VCC)
- net 22M-13: no longer 22M1.13 (B5)
- net EXP-A10: now also U71.1 (M1), 26E.1 (~R), 26E.13 (~R)
- net GND: now also U71.15 (TDI), U71.16 (TMS), U71.17 (TCK), U71.30 (TDO); no longer 13E1.91
- net IO-ADDR-18: now also U71.14 (M12)
- net IO-ADDR-19: now also U71.13 (M11)
- net IO-ADDR-20: now also U71.12 (M10)
- net IO-ADDR-21: now also U71.11 (M9)
- net IO-DATA-0: now also 26E.2 (D)
- net IO-DATA-8: now also 26E.12 (D)
- net U17-4: no longer U71.4 (M4)
- net U71-27: now reaches 13E1.100
- net U71-27: now also U71.27 (M15), 26E.11 (C)
- net 18E-35: now reaches 13E1.95
- net 18E-36: now reaches 13E1.96
- net 35J-5: now reaches 13E1.97
- net BUS-~RD: now reaches U71.18 (M13)
- net PSX-~BIOS: now reaches U71.19 (M14)
- net U71-2: now reaches U71.2 (M1)
- net U71-22: now reaches U71.22 (M16)
- net U71-24: now reaches U71.24 (M17)
- net U71-24: now also 22M1.13 (B5)
- net U71-26: now reaches U71.26 (M16)
- net U71-29: now reaches U71.29 (M13)
- net U71-29: now also 26E.3 (C)
- net U71-3: now reaches U71.3 (M2)
- net U71-34: now reaches U71.34 (M11)
- net U71-37: now reaches U71.37 (M8)
- net U71-40: now reaches U71.40 (I/O/GTS2)
- net U71-44: now reaches U71.44 (M2)
- net ADC-CLK: no longer names the net of 13E1.80
- net KCUS-98 renamed 35J-9
- net NVRAM-~WR renamed BUS-~WR
- net U17-6 renamed U71-6
- net U17-7 renamed U71-7
- net U71-33: no longer names the net of U71.33 (M12)
- new net +3V3: 22M1.20 (VCC), 22N1.20 (VCC), 22Q1.20 (VCC)
- new net 18E-10: 26E.9 (Q)
- new net IDE-~RST: 26E.5 (Q)
- new net U71-4: U71.4 (M4)
Other:
- note added: "21C-13 H8 Control Pin"
- note added: "21C-5 near H8"
- note added: "24E\n1-6: No connect\n8-11: JVS Sense trigger and logic input\n12-13: Cart pin 28 and 20 shenanigans"
- note added: "26E-11 H8 Reset toggle"
- note added: "26E-3 IDE Reset toggle"
- note added: "35J-1 Reset A"
- note added: "BIOS-~OE"
- note added: "Cart 27"
- note added: "Cart 31"
- note added: "EXT-OUT Latch clock"
- note added: "Expansion IO"
- note added: "Flash/PCMCIA Memory select"
- note added: "Holds the H8 in reset until activated"
- note added: "Holds the IDE bus in reset until activated"
- note added: "IDE Bus CE"
- note added: "IDE INT Request"
- note added: "IDE-CS0\nIDE-CS1"
- note added: "IRQ10 Output"
- note added: "JVS Buffer has data"
- note added: "JVS Sense line"
- note added: "Konami Custom 102"
- note added: "RTC OE"
- note added: "Watchdog kick"
- note removed: "27F CP"
- note removed: "Slot-0 PCMCIA CE Stuff"
- moved on the sheet: 13E1G, 13E1H, 13E1J, 13E2K, 22D1, 22E1, 22M1, 22N1, 22Q1, 23L1, 25T1, 27F1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

Commit message: Added 3D Models
Connections:
- net U71-38: now reaches U71.38 (M7)
- net CART-28 renamed KCUS-93
Other:
- note added: "Cart 28"
- note added: "Security Cart Pin 30?"
Changed lines of the file:
@@
 35J-9
 Text GLabel 5550 7350 0    50   Input ~ 0
-CART-28
+KCUS-93
 Text Notes 12600 7600 0    50   ~ 0
 24E\n1-6: No connect\n8-11: JVS Sense trigger and logic input\n12-13: Cart pin 28 and 20 shenanigans
@@
 Wire Wire Line
 	17150 5100 17250 5100
+Text Notes 15100 6050 0    50   ~ 0
+Expansion IO
+Text GLabel 23150 4850 2    50   Input ~ 0
+U71-38
+Wire Wire Line
+	23150 4850 22950 4850
 Wire Bus Line
 	4950 9800 7900 9800
@@
 Wire Bus Line
 	1550 1350 1550 6500
-Text Notes 15100 6050 0    50   ~ 0
-Expansion IO
+Text Notes 23550 4900 0    50   ~ 0
+Security Cart Pin 30?
+Text Notes 5050 7400 2    50   ~ 0
+Cart 28
 $EndSCHEMATC
