File: Schematics/Security-cart.sch (KiCad schematic (older format))
At the start: 11 parts, among them CN4 SECURITY_CART

Commit message: Added 3D Models
Parts:
- removed 35J1: 74LS125, Package_SO:SO-14_3.9x8.65mm_P1.27mm, symbol 74xx:74LS125
Connections:
- net 35J-5: no longer CN4.31 (Pin_31)
- net ~RESET: now also CN4.7 (Pin_7)
- net 35J-11 renamed U71-38
- net CART-28 renamed KCUS-93
- new net KCUS-97: CN4.31 (Pin_31)
Other:
- note added: "No connect?"
- moved on the sheet: 24E?F, 35H1B, 35H?C, 35JA, 35JB
