File: Schematics (KiCad)/GX700-PWB/Ksys573.kicad_pcb (KiCad board)
At the start: 4 copper layers, 295 x 285 mm, 105 parts, among them CN1 B6P-VH, CN15 B4P-VH, CN2 VGA-DSUB15, CN2I1 ATA-IDE, CN5 B12PSHF1A, U1 KONAMI-058232, U2 ADC0834, U3 74LS74, U4 M48T58Y, U71 22J-X700A1 XC9536

Commit message: Added Symbols, PSX page
Added PSX CPU and GPU symbols, added a COH PSX skeleton schematic and also updated the JAMMA symbol and footprint as it was bad.
Parts:
- added 13E1: KONAMI_056879, Package_QFP:TQFP-120_14x14mm_P0.4mm, F.Cu at (436.9, 289.6)
- added 13E2: KONAMI_056879, Package_QFP:TQFP-120_14x14mm_P0.4mm, F.Cu at (454.8, 289.6)
- added 13E3: KONAMI_056879, Package_QFP:TQFP-120_14x14mm_P0.4mm, F.Cu at (562.4, 272.2)
- added 22D1: 74LS273, Package_SO:SO-20_5.3x12.6mm_P1.27mm, F.Cu at (469.0, 301.8)
- added 22E1: 74LS273, Package_SO:SO-20_5.3x12.6mm_P1.27mm, F.Cu at (469.0, 287.7)
- added 24E2: 74LS14, Package_SO:SO-14_3.9x8.65mm_P1.27mm, F.Cu at (440.6, 320.2)
- added 25T1: S240, Connector_PinHeader_2.54mm:PinHeader_2x04_P2.54mm_Vertical, F.Cu at (478.9, 317.4)
- added 26E1: 74LS74, Package_SO:SO-14_5.3x10.2mm_P1.27mm, F.Cu at (513.6, 269.1)
- added 27F1: 74LS273, Package_SO:SO-20_5.3x12.6mm_P1.27mm, F.Cu at (534.9, 287.7)
- added 29G2: 74LS139, Package_SO:SOIC-16_4.55x10.3mm_P1.27mm, F.Cu at (571.1, 239.9)
- added 31A1: LINE L-OUT, Arcade:RCA, F.Cu at (412.9, 102.9)
- added 32D1: SM5877AM, Package_SO:SSOP-24_5.3x8.2mm_P0.65mm, F.Cu at (523.3, 244.1)
- added 33A1: LINE R-OUT, Arcade:RCA, F.Cu at (412.9, 117.8)
- added 35H1: 74LS125, Package_SO:SO-14_3.9x8.65mm_P1.27mm, F.Cu at (432.1, 320.2)
- added 35H2: 74LS125, Package_SO:SO-14_3.9x8.65mm_P1.27mm, F.Cu at (449.0, 320.2)
- added 35J1: 74LS74, Package_SO:SO-14_3.9x8.65mm_P1.27mm, F.Cu at (432.1, 330.4)
- added 36A1: ZBDS5101-8PT, Package_SO:SOIC-16_4.55x10.3mm_P1.27mm, F.Cu at (360.7, 104.1)
- added 36A1: ZBDS5101-8PT, Package_SO:SOIC-16_4.55x10.3mm_P1.27mm, F.Cu at (342.9, 104.1)
- added C12: 10n, Capacitor_SMD:C_0805_2012Metric, F.Cu at (434.6, 300.0)
- added C13: 10n, Capacitor_SMD:C_0805_2012Metric, F.Cu at (430.1, 300.0)
- added C158: 10M16E, Capacitor_THT:CP_Radial_D5.0mm_P2.50mm, F.Cu at (503.4, 306.7)
- added C6/5B1: EMI222, Connector_PinHeader_2.54mm:PinHeader_1x03_P2.54mm_Vertical, F.Cu at (547.1, 282.9)
- added CN2: VGA-DSUB15, Connector_Dsub:DSUB-15-HD_Female_Horizontal_P2.29x1.98mm_EdgePinOffset8.35mm_Housed_MountingHolesOffset10.89mm, F.Cu at (517.5, 283.7)
- added CN22: BS4PSHF1AA, Connector_PinHeader_2.54mm:PinHeader_1x04_P2.54mm_Vertical, F.Cu at (443.2, 86.4)
- added CPU1: CXD8530CQ, Package_QFP:LQFP-208_28x28mm_P0.5mm, F.Cu at (476.5, 250.2)
- added GPU1: CXD8561CQ, Package_QFP:LQFP-208_28x28mm_P0.5mm, F.Cu at (444.1, 250.2)
- added JP5: Jumper_NO_Small, Connector_PinSocket_2.54mm:PinSocket_1x02_P2.54mm_Vertical, F.Cu at (499.1, 305.8)
- added LA4705: LA4705, Package_SIP:SIP18_Housing, F.Cu at (510.1, 236.5)
- added R83: 220, Resistor_SMD:R_0805_2012Metric_Pad1.20x1.40mm_HandSolder, F.Cu at (435.0, 275.9)
- added R84: 220, Resistor_SMD:R_0805_2012Metric_Pad1.20x1.40mm_HandSolder, F.Cu at (439.8, 275.9)
- added R85: 220, Resistor_SMD:R_0805_2012Metric_Pad1.20x1.40mm_HandSolder, F.Cu at (446.7, 267.9)
- added R86: 220, Resistor_SMD:R_0805_2012Metric_Pad1.20x1.40mm_HandSolder, F.Cu at (495.1, 243.4)
- added R87: 220, Resistor_SMD:R_0805_2012Metric_Pad1.20x1.40mm_HandSolder, F.Cu at (430.3, 275.9)
- added RA10: 472, Resistor_SMD:R_Array_Convex_5x1206, F.Cu at (495.5, 238.0)
- added RA11: 472, Resistor_SMD:R_Array_Convex_5x1206, F.Cu at (441.6, 270.4)
- added RA27: 4.7k, Resistor_SMD:R_Array_Convex_5x1206, F.Cu at (439.1, 329.2)
- added RA8: 472, Resistor_SMD:R_Array_Convex_5x1206, F.Cu at (430.6, 270.4)
- added RA9: 472, Resistor_SMD:R_Array_Convex_5x1206, F.Cu at (436.1, 270.4)
- added S86: Conn_01x03, Connector_PinHeader_2.54mm:PinHeader_1x03_P2.54mm_Vertical, F.Cu at (542.5, 282.9)
- added U1: L78L05_SOT89, Package_TO_SOT_SMD:SOT-89-3, F.Cu at (558.2, 237.0)
- CN1: renamed from EXT-IN-CN1; value Conn_01x10_Male -> B10PSHF1A
- CN3: renamed from ANALOG-CN1; value Conn_01x10_Male -> B10PSHF1A
- renumbered U1 to 058232/58460, CN1 to CN17, RA9 to RA25, RA8 to RA26
Connections:
- net 21C-11 renamed 18E-54
- net EXT-IN-10 renamed Net-(15B2-Pad8)
- net EXT-IN-3 renamed J1-B4
- net EXT-IN-5 renamed Net-(15B2-Pad3)
- net EXT-IN-6 renamed Net-(15B2-Pad4)
- net JV-GND renamed Net-(10B1-Pad4)
- net Net-(18E1-Pad10) renamed H8-~{RST}
- net Net-(18E1-Pad16) renamed 18E-16
- net Net-(18E1-Pad55) renamed 18E-55
- net Net-(18E1-Pad56) renamed 18E-56
- net Net-(18E1-Pad57) renamed 18E-57
- net Net-(U71-Pad29) renamed U71-29
- net Net-(U71-Pad36) renamed ~{EXP2}
- net Net-(U71-Pad6) renamed U71-6
- net U17-7 renamed U71-7
- 058232/58460 pad 13: EXP-A10 -> ~{RESET}
- 058232/58460 pad 14: (no net) -> unconnected-(058232/58460-Pad14)
- 058232/58460 pad 8: +5V -> Net-(058232/58460-Pad8)
- 058232/58460 pad 9: U71-43 -> WD_KICK
- 10B1 pad 14: Net-(10B1-Pad14) -> unconnected-(10B1-Pad14)
- 10B1 pad 3: Net-(10B1-Pad3) -> unconnected-(10B1-Pad3)
- 10S1 pad 1: IDE-AB -> BUS-~{RD}
- 10S1 pad 19: IDE-CE -> U71-34
- 10S1 pad 20: +5V -> IO-ADDR-10
- 12S1 pad 1: IDE-AB -> BUS-~{RD}
- 12S1 pad 19: IDE-CE -> U71-34
- 12S1 pad 20: +5V -> IO-ADDR-10
- 12S1 pad 8: /IDE/IO-DATA-0 -> IO-DATA-0
- 13T1 pad 15: /IDE/IDE-CS0 -> IDE-CS0
- 13T1 pad 16: /IDE/IDE-CS1 -> IDE-CS1
- 14S1 pad 1: +5V -> IO-ADDR-10
- 14S1 pad 2: EXP-A10 -> IDE-~{RST}
- 14S1 pad 20: +5V -> IO-ADDR-10
- 14S1 pad 8: U17-2 -> IDE-CS0
- 14S1 pad 9: U17-3 -> IDE-CS1
- 15B1 pad 15: +5V -> IO-ADDR-10
- 15B1 pad 16: +5V -> IO-ADDR-10
- 15B2 pad 2: EXT-IN-4 -> J1-B5
- 15B2 pad 5: EXT-IN-7 -> J2-B4
- 15B2 pad 6: EXT-IN-8 -> Net-(15B2-Pad6)
- 15B2 pad 7: EXT-IN-9 -> J2-B5
- 18E1 pad 19: Net-(13E1-Pad51) -> Net-(13E1-Pad52)
- 18E1 pad 20: Net-(13E1-Pad52) -> Net-(13E1-Pad53)
- 18E1 pad 21: Net-(13E1-Pad53) -> Net-(13E1-Pad54)
- 18E1 pad 22: Net-(13E1-Pad54) -> Net-(13E1-Pad55)
- 18E1 pad 23: Net-(13E1-Pad55) -> Net-(13E1-Pad56)
- 18E1 pad 24: Net-(13E1-Pad56) -> Net-(13E1-Pad57)
- 18E1 pad 25: 18E-25 -> Net-(13E2-Pad39)
- 18E1 pad 26: 18E-26 -> Net-(13E2-Pad40)
- 18E1 pad 33: +5V -> IO-ADDR-10
- 18E1 pad 58: +5V -> IO-ADDR-10
- 18E1 pad 6: +5V -> IO-ADDR-10
- 18E1 pad 9: Net-(18E1-Pad9) -> unconnected-(18E1-Pad9)
- 20C1 pad 8: +5V -> IO-ADDR-10
- 21C1 pad 10: +5V -> IO-ADDR-10
- 21C1 pad 12: +5V -> IO-ADDR-10
- 21C1 pad 2: +5V -> IO-ADDR-10
- 21C1 pad 3: 22E-CP -> H8-TX-FLAG
- 21C1 pad 4: +5V -> IO-ADDR-10
- 21C1 pad 6: Net-(21C1-Pad6) -> unconnected-(21C1-Pad6)
- 21C1 pad 8: Net-(21C1-Pad8) -> unconnected-(21C1-Pad8)
- 22G1 pad 1: +5V -> IO-ADDR-10
- 22G1 pad 24: PCPU-~{BIOS} -> PSX-~{BIOS}
- 22G1 pad 32: +5V -> IO-ADDR-10
- 22M1 pad 11: EXP-A10 -> ~{RESET}
- 22M1 pad 13: 22M-13 -> U71-24
- 22M1 pad 2: Net-(22M1-Pad2) -> unconnected-(22M1-Pad2)
- 22M1 pad 20: +5V -> +3V3
- 22M1 pad 3: Net-(22M1-Pad3) -> unconnected-(22M1-Pad3)
- 22N1 pad 11: /IO-DATA-7 -> IO-DATA-7
- 22N1 pad 12: /IO-DATA-6 -> IO-DATA-6
- 22N1 pad 13: /IO-DATA-5 -> IO-DATA-5
- 22N1 pad 14: /IO-DATA-4 -> IO-DATA-4
- 22N1 pad 15: /IO-DATA-3 -> IO-DATA-3
- 22N1 pad 16: /IO-DATA-2 -> IO-DATA-2
- 22N1 pad 17: /IO-DATA-1 -> IO-DATA-1
- 22N1 pad 18: /IO-DATA-0 -> IO-DATA-0
- 22N1 pad 19: U17-35 -> ~{DBUS-EN}
- 22N1 pad 20: +5V -> +3V3
- 22Q1 pad 11: /IO-DATA-15 -> IO-DATA-15
- 22Q1 pad 12: /IO-DATA-14 -> IO-DATA-14
- 22Q1 pad 13: /IO-DATA-13 -> IO-DATA-13
- 22Q1 pad 14: /IO-DATA-12 -> IO-DATA-12
- 22Q1 pad 15: /IO-DATA-11 -> IO-DATA-11
- 22Q1 pad 16: /IO-DATA-10 -> IO-DATA-10
- 22Q1 pad 17: /IO-DATA-9 -> IO-DATA-9
- 22Q1 pad 18: /IO-DATA-8 -> IO-DATA-8
- 22Q1 pad 19: U17-35 -> ~{DBUS-EN}
- 22Q1 pad 20: +5V -> +3V3
- 23L1 pad 1: +5V -> IO-ADDR-10
- 23L1 pad 2: Net-(23L1-Pad2) -> unconnected-(23L1-Pad2)
- 23L1 pad 20: +5V -> IO-ADDR-10
- 23L1 pad 3: Net-(23L1-Pad3) -> unconnected-(23L1-Pad3)
- 23L1 pad 4: Net-(23L1-Pad4) -> unconnected-(23L1-Pad4)
- 25B1 pad 11: +5V -> IO-ADDR-10
- 25R1 pad 1: U17-33 -> ~{PCMCIA_CE1}
- 26D1 pad 1: +5V -> IO-ADDR-10
- 27G1 pad 13: /IO-DATA-4 -> IO-DATA-4
- 27G1 pad 14: /IO-DATA-5 -> IO-DATA-5
- 27G1 pad 17: /IO-DATA-6 -> IO-DATA-6
- 27G1 pad 18: /IO-DATA-7 -> IO-DATA-7
- 27G1 pad 20: +5V -> IO-ADDR-10
- 27G1 pad 3: /IO-DATA-0 -> IO-DATA-0
- 27G1 pad 4: /IO-DATA-1 -> IO-DATA-1
- 27G1 pad 7: /IO-DATA-2 -> IO-DATA-2
- 27G1 pad 8: /IO-DATA-3 -> IO-DATA-3
- 27H1 pad 12: +5V -> IO-ADDR-10
- 27H1 pad 14: EXP-A10 -> ~{RESET}
- 27H1 pad 37: +5V -> IO-ADDR-10
- 27H1 pad 42: Net-(27H1-Pad42) -> unconnected-(27H1-Pad42)
- 27J1 pad 12: +5V -> IO-ADDR-10
- 27J1 pad 14: EXP-A10 -> ~{RESET}
- 27J1 pad 37: +5V -> IO-ADDR-10
- 27J1 pad 42: Net-(27J1-Pad42) -> unconnected-(27J1-Pad42)
- 27L1 pad 12: +5V -> IO-ADDR-10
- 27L1 pad 14: EXP-A10 -> ~{RESET}
- 27L1 pad 37: +5V -> IO-ADDR-10
- 27L1 pad 42: Net-(27L1-Pad42) -> unconnected-(27L1-Pad42)
- 27M1 pad 12: +5V -> IO-ADDR-10
- 27M1 pad 14: EXP-A10 -> ~{RESET}
- 27M1 pad 37: +5V -> IO-ADDR-10
- 27M1 pad 42: Net-(27M1-Pad42) -> unconnected-(27M1-Pad42)
- 27N1 pad 1: +5V -> IO-ADDR-10
- 27N1 pad 20: +5V -> IO-ADDR-10
- 28E1 pad 1: EXT-OUTPUT-7 -> Net-(27F1-Pad19)
- 28E1 pad 11: EXT-OUTPUT-4 -> Net-(27F1-Pad12)
- 28E1 pad 13: EXT-OUTPUT-6 -> Net-(27F1-Pad16)
- 28E1 pad 3: EXT-OUTPUT-5 -> Net-(27F1-Pad15)
- 28E1 pad 5: EXT-OUTPUT-3 -> Net-(27F1-Pad9)
- 28E1 pad 9: EXT-OUTPUT-2 -> Net-(27F1-Pad6)
- 29E1 pad 1: EXT-OUTPUT-0 -> Net-(27F1-Pad2)
- 29E1 pad 10: Net-(29E1-Pad10) -> unconnected-(29E1-Pad10)
- 29E1 pad 11: Net-(29E1-Pad11) -> unconnected-(29E1-Pad11)
- 29E1 pad 13: EXT-OUTPUT-1 -> Net-(27F1-Pad5)
- 29E1 pad 3: Net-(29E1-Pad3) -> unconnected-(29E1-Pad3)
- 29E1 pad 4: Net-(29E1-Pad4) -> unconnected-(29E1-Pad4)
- 29E1 pad 5: Net-(29E1-Pad5) -> unconnected-(29E1-Pad5)
- 29E1 pad 6: Net-(29E1-Pad6) -> unconnected-(29E1-Pad6)
- 29E1 pad 8: Net-(29E1-Pad8) -> unconnected-(29E1-Pad8)
- 29E1 pad 9: Net-(29E1-Pad9) -> unconnected-(29E1-Pad9)
- 30N1 pad 1: +5V -> IO-ADDR-10
- 30N1 pad 18: IO-ADDR-8 -> IO-ADDR-10
- 30N1 pad 20: +5V -> IO-ADDR-10
- 31H1 pad 12: +5V -> IO-ADDR-10
- 31H1 pad 14: EXP-A10 -> ~{RESET}
- 31H1 pad 37: +5V -> IO-ADDR-10
- 31H1 pad 42: Net-(31H1-Pad42) -> unconnected-(31H1-Pad42)
- 31J1 pad 12: +5V -> IO-ADDR-10
- 31J1 pad 14: EXP-A10 -> ~{RESET}
- 31J1 pad 37: +5V -> IO-ADDR-10
- 31J1 pad 42: Net-(31J1-Pad42) -> unconnected-(31J1-Pad42)
- 31L1 pad 12: +5V -> IO-ADDR-10
- 31L1 pad 14: EXP-A10 -> ~{RESET}
- 31L1 pad 37: +5V -> IO-ADDR-10
- 31L1 pad 42: Net-(31L1-Pad42) -> unconnected-(31L1-Pad42)
- 31M1 pad 12: +5V -> IO-ADDR-10
- 31M1 pad 14: EXP-A10 -> ~{RESET}
- 31M1 pad 37: +5V -> IO-ADDR-10
- 31M1 pad 42: Net-(31M1-Pad42) -> unconnected-(31M1-Pad42)
- 32N1 pad 1: +5V -> IO-ADDR-10
- 32N1 pad 20: +5V -> IO-ADDR-10
- 35K1 pad 1: EXP-A10 -> ~{RESET}
- 35K1 pad 2: Net-(35K1-Pad2) -> CART-20
- 35K1 pad 20: +5V -> IO-ADDR-10
- 5T1 pad 1: +5V -> IO-ADDR-10
- C209 pad 1: +5V -> IO-ADDR-10
- C38 pad 1: +5V -> IO-ADDR-10
- C39 pad 1: +5V -> IO-ADDR-10
- C40 pad 1: +5V -> IO-ADDR-10
- C43 pad 1: +5V -> IO-ADDR-10
- CN1 pad 1: +5V -> IO-ADDR-10
- CN1 pad 2: +5V -> IO-ADDR-10
- CN1 pad 4: EXT-IN-4 -> J1-B5
- CN1 pad 7: EXT-IN-7 -> J2-B4
- CN1 pad 8: EXT-IN-8 -> Net-(15B2-Pad6)
- CN1 pad 9: EXT-IN-9 -> J2-B5
- CN17 pad 1: +5V -> IO-ADDR-10
- CN17 pad 2: +5V -> IO-ADDR-10
- CN2I1 pad 20: Net-(CN2I1-Pad20) -> unconnected-(CN2I1-Pad20)
- CN2I1 pad 31: Net-(CN2I1-Pad31) -> U71-22
- CN2I1 pad 32: Net-(CN2I1-Pad32) -> unconnected-(CN2I1-Pad32)
- CN2I1 pad 34: Net-(CN2I1-Pad34) -> unconnected-(CN2I1-Pad34)
- CN2I1 pad 37: /IDE/IDE-CS0 -> IDE-CS0
- CN2I1 pad 38: /IDE/IDE-CS1 -> IDE-CS1
- CN2I1 pad 39: Net-(CN2I1-Pad39) -> unconnected-(CN2I1-Pad39)
- CN3 pad 1: +5V -> IO-ADDR-10
- CN3 pad 2: +5V -> IO-ADDR-10
- DIPSW4P1 pad 1: Net-(DIPSW4P1-Pad1) -> GND
- EXO-1 pad 1: Net-(EXO-1-Pad1) -> unconnected-(EXO-1-Pad1)
- EXO-1 pad 3: +5V -> IO-ADDR-10
- EXO-1 pad 8: +5V -> IO-ADDR-10
- JAMMA1 pad A10: Net-(JAMMA1-PadA10) -> unconnected-(JAMMA1-PadA10)
- JAMMA1 pad A25: EXT-IN-7 -> J1-B5
- JAMMA1 pad A4: Net-(5B1-Pad3) -> Net-(4B1-Pad3)
- JAMMA1 pad A5: Net-(JAMMA1-PadA5) -> Net-(5B1-Pad3)
- JAMMA1 pad B10: Net-(JAMMA1-PadB10) -> unconnected-(JAMMA1-PadB10)
- JAMMA1 pad B13: VGA-CSYNC -> Net-(10B1-Pad6)
- JAMMA1 pad B14: Net-(JAMMA1-PadB14) -> unconnected-(JAMMA1-PadB14)
- JAMMA1 pad B24: EXT-IN-4 -> J2-B4
- JAMMA1 pad B25: EXT-IN-8 -> J2-B5
- JAMMA1 pad B4: Net-(5B1-Pad3) -> Net-(4B1-Pad3)
- JAMMA1 pad B5: Net-(JAMMA1-PadB5) -> Net-(5B1-Pad3)
- R289 pad 1: +5V -> IO-ADDR-10
- RA1 pad 10: +5V -> IO-ADDR-10
- RA1 pad 5: +5V -> IO-ADDR-10
- RA2 pad 10: +5V -> IO-ADDR-10
- RA2 pad 5: +5V -> IO-ADDR-10
- RA25 pad 10: +5V -> IO-ADDR-10
- RA25 pad 5: +5V -> IO-ADDR-10
- RA26 pad 10: +5V -> IO-ADDR-10
- RA26 pad 5: +5V -> IO-ADDR-10
- RA26 pad 6: CART-27 -> 35J-9
- RA3 pad 1: Net-(RA3-Pad1) -> unconnected-(RA3-Pad1)
- RA3 pad 10: +5V -> IO-ADDR-10
- RA3 pad 5: +5V -> IO-ADDR-10
- RA3 pad 9: Net-(RA3-Pad9) -> unconnected-(RA3-Pad9)
- RA4 pad 1: Net-(RA4-Pad1) -> unconnected-(RA4-Pad1)
- RA4 pad 2: Net-(RA4-Pad2) -> unconnected-(RA4-Pad2)
- RA4 pad 3: Net-(RA4-Pad3) -> unconnected-(RA4-Pad3)
- RA4 pad 5: +5V -> IO-ADDR-10
- RA5 pad 10: +5V -> IO-ADDR-10
- RA5 pad 5: +5V -> IO-ADDR-10
- RA6 pad 10: +5V -> IO-ADDR-10
- RA6 pad 5: +5V -> IO-ADDR-10
- RA6 pad 6: IO-ADDR-8 -> IO-ADDR-10
- RA7 pad 10: +5V -> IO-ADDR-10
- RA7 pad 5: +5V -> IO-ADDR-10
- U2 pad 1: Net-(U2-Pad1) -> unconnected-(U2-Pad1)
- U2 pad 14: +5V -> IO-ADDR-10
- U2 pad 9: +5V -> IO-ADDR-10
- U4 pad 1: Net-(U4-Pad1) -> RTC-FT
- U4 pad 10: Net-(U4-Pad10) -> unconnected-(U4-Pad10)
- U4 pad 2: Net-(U4-Pad2) -> unconnected-(U4-Pad2)
- U4 pad 20: Net-(U4-Pad20) -> RTC-OE
- U4 pad 21: Net-(U4-Pad21) -> unconnected-(U4-Pad21)
- U4 pad 22: Net-(U4-Pad22) -> BUS-~{RD}
- U4 pad 23: Net-(U4-Pad23) -> unconnected-(U4-Pad23)
- U4 pad 24: Net-(U4-Pad24) -> unconnected-(U4-Pad24)
- U4 pad 25: Net-(U4-Pad25) -> unconnected-(U4-Pad25)
- U4 pad 26: +5V -> IO-ADDR-10
- U4 pad 27: NVRAM-~{WR} -> BUS-~{WR}
- U4 pad 28: +5V -> IO-ADDR-10
- U4 pad 3: Net-(U4-Pad3) -> unconnected-(U4-Pad3)
- U4 pad 4: Net-(U4-Pad4) -> unconnected-(U4-Pad4)
- U4 pad 5: Net-(U4-Pad5) -> unconnected-(U4-Pad5)
- U4 pad 6: Net-(U4-Pad6) -> unconnected-(U4-Pad6)
- U4 pad 7: Net-(U4-Pad7) -> unconnected-(U4-Pad7)
- U4 pad 8: Net-(U4-Pad8) -> unconnected-(U4-Pad8)
- U4 pad 9: Net-(U4-Pad9) -> unconnected-(U4-Pad9)
- U71 pad 1: Net-(U71-Pad1) -> ~{RESET}
- U71 pad 11: Net-(U71-Pad11) -> IO-ADDR-21
- U71 pad 12: Net-(U71-Pad12) -> IO-ADDR-20
- U71 pad 13: Net-(U71-Pad13) -> IO-ADDR-19
- U71 pad 14: Net-(U71-Pad14) -> IO-ADDR-18
- U71 pad 15: Net-(U71-Pad15) -> GND
- U71 pad 16: Net-(U71-Pad16) -> GND
- U71 pad 17: Net-(U71-Pad17) -> GND
- U71 pad 18: Net-(U71-Pad18) -> BUS-~{RD}
- U71 pad 19: Net-(U71-Pad19) -> PSX-~{BIOS}
- U71 pad 2: Net-(U71-Pad2) -> IDE-CS0
- U71 pad 20: Net-(U71-Pad20) -> IO-ADDR-10
- U71 pad 21: +5V -> IO-ADDR-10
- U71 pad 22: Net-(U71-Pad22) -> U71-22
- U71 pad 24: Net-(U71-Pad24) -> U71-24
- U71 pad 25: NVRAM-~{WR} -> BUS-~{WR}
- U71 pad 26: Net-(U71-Pad26) -> U71-26
- U71 pad 27: Net-(U71-Pad27) -> U71-27
- U71 pad 28: Net-(U71-Pad28) -> ~{EXP1}
- U71 pad 3: Net-(U71-Pad3) -> IDE-CS1
- U71 pad 30: Net-(U71-Pad30) -> GND
- U71 pad 32: +5V -> IO-ADDR-10
- U71 pad 33: U71-33 -> ~{PCMCIA_CE1}
- U71 pad 34: Net-(U71-Pad34) -> U71-34
- U71 pad 35: Net-(U71-Pad35) -> ~{DBUS-EN}
- U71 pad 37: Net-(U71-Pad37) -> ~{PCMCIA_CE2}
- U71 pad 38: Net-(U71-Pad38) -> U71-38
- U71 pad 39: U71-39 -> H8-TX-FLAG
- U71 pad 4: U17-4 -> U71-4
- U71 pad 40: Net-(U71-Pad40) -> RTC-OE
- U71 pad 41: +5V -> IO-ADDR-10
- U71 pad 42: Net-(U71-Pad42) -> ~{EXP-CE}
- U71 pad 43: U71-43 -> EXT-OUT-LATCH
- U71 pad 44: Net-(U71-Pad44) -> WD_KICK
Routing:
- net Net-(24A1-Pad5): vias 0 -> 1
- net (no net): vias 0 -> 1
