File: Schematics (KiCad)/GX700-PWB/573-IDE.kicad_sch (KiCad schematic)
At the start: 21 parts, among them CN15 B4P-VH, CN2I1 ATA-IDE, CN2P1 Intergrated IDE Connector

Commit message: Added Symbols, PSX page
Added PSX CPU and GPU symbols, added a COH PSX skeleton schematic and also updated the JAMMA symbol and footprint as it was bad.
Parts:
- gave numbers to parts that had none: 1
Changed lines of the file:
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@@
   (symbol (lib_id "power:+5V") (at 62.23 139.7 0) (unit 1)
     (in_bom yes) (on_board yes)
-    (property "Reference" "#PWR?" (id 0) (at 62.23 143.51 0)
+    (property "Reference" "#PWR0267" (id 0) (at 62.23 143.51 0)
       (effects (font (size 1.27 1.27)) hide)
     )
@@
   (symbol (lib_id "74xx:74LS74") (at 62.23 147.32 0) (unit 1)
     (in_bom yes) (on_board yes)
-    (property "Reference" "26E?" (id 0) (at 68.58 137.16 0))
+    (property "Reference" "26E1" (id 0) (at 68.58 137.16 0))
     (property "Value" "74LS74" (id 1) (at 68.58 139.7 0))
     (property "Footprint" "Package_SO:SO-14_5.3x10.2mm_P1.27mm" (id 2) (at 62.23 147.32 0)

Commit message: General Fixes
Connections:
- net U71-34 renamed ~{IDE-CE}
Changed lines of the file:
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@@
     )
   )
-  (global_label "U71-34" (shape input) (at 50.8 66.04 180) (fields_autoplaced)
+  (global_label "~{IDE-CE}" (shape input) (at 50.8 66.04 180) (fields_autoplaced)
     (effects (font (size 1.27 1.27)) (justify right))
     (property "Intersheet References" "${INTERSHEET_REFS}" (id 0) (at -6.35 2.54 0)
@@
     )
   )
-  (global_label "IDE-~{RST}" (shape input) (at 73.66 144.78 0) (fields_autoplaced)
+  (global_label "IDE-~{RST}" (shape output) (at 73.66 144.78 0) (fields_autoplaced)
     (effects (font (size 1.27 1.27)) (justify left))
-    (property "Intersheet References" "${INTERSHEET_REFS}" (id 0) (at -3.81 -96.52 0)
-      (effects (font (size 1.27 1.27)) hide)
+    (property "Intersheet References" "${INTERSHEET_REFS}" (id 0) (at 84.0275 144.7006 0)
+      (effects (font (size 1.27 1.27)) (justify left) hide)
     )
   )

Commit message: Major board changes to give a rough render of the PCB
Parts:
- CN2I1: footprint Connector_PinSocket_2.54mm:PinSocket_2x20_P2.54mm_Vertical -> Connector_PinHeader_2.54mm:PinHeader_2x20_P2.54mm_Vertical
Connections:
- net at 13T1.1: now also 14S1.18 (B0); no longer 14S1.11 (B7)
- net at 13T1.2: now also 14S1.17 (B1); no longer 14S1.12 (B6)
- net at 13T1.3: now also 14S1.16 (B2); no longer 14S1.13 (B5)
- net at 13T1.4: now also 14S1.15 (B3); no longer 14S1.14 (B4)
- net at 13T1.5: now also 14S1.14 (B4); no longer 14S1.15 (B3)
- net at 13T1.6: now also 14S1.13 (B5); no longer 14S1.16 (B2)
- net at 13T1.7: now also 14S1.12 (B6); no longer 14S1.17 (B1)
- net at 13T1.8: now also 14S1.11 (B7); no longer 14S1.18 (B0)
Other:
- moved on the sheet: 13T1
