File: Schematics (KiCad)/GX700-PWB/573-PCCARD.kicad_sch (KiCad schematic)
At the start: 4 parts

Commit message: Added Symbols, PSX page
Added PSX CPU and GPU symbols, added a COH PSX skeleton schematic and also updated the JAMMA symbol and footprint as it was bad.
Parts:
- gave numbers to parts that had none: 1
Changed lines of the file:
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@@
   (symbol (lib_id "74xx:74LS139") (at 57.15 162.56 0) (unit 1)
     (in_bom yes) (on_board yes)
-    (property "Reference" "29G?" (id 0) (at 57.15 153.2382 0))
+    (property "Reference" "29G2" (id 0) (at 57.15 153.2382 0))
     (property "Value" "74LS139" (id 1) (at 57.15 155.5496 0))
     (property "Footprint" "Package_SO:SOIC-16_4.55x10.3mm_P1.27mm" (id 2) (at 57.15 162.56 0)

Commit message: General Fixes
Connections:
- net IO-AD-0 is gone; now on net IO-ADDR-0: 25S1.2 (Pin_2), 25S1.3 (Pin_3)
- net IO-AD-16 is gone; now on net IO-ADDR-16: 25S1.1 (Pin_1)
- net 27G-12 renamed FBANK-A0
- net 27G-15 renamed FBANK-A1
- net 27G-2 renamed PCCD-A22
- net 27G-5 renamed PCCD-A23
- net 27G-6 renamed PCCD-A24
- net 27G-9 renamed PCCD-A25
Other:
- note added: "Cut 2-3 Link and jumper 1-2 to enable CE1 for CF cards"
- note added: "Flash/CF Card Selection"
- note added: "Latched AD Lines from 27G"
- note added: "Only exists on rev. C and above"
- note removed: "CE Selection Jumper?"
- note removed: "Cut 2-3 Link and jumper 1-2 to enable CE1?"
- note removed: "Latched AD Lines"

Commit message: Major board changes to give a rough render of the PCB
Parts:
- renumbered 29G2 to 29G1
