File: Schematics (KiCad)/GX700-PWB/573-ROM.kicad_sch (KiCad schematic)
At the start: 11 parts, among them U4 M48T58Y

Commit message: General Fixes
Connections:
- net 27G-2 renamed PCCD-A22
- net 27G-5 renamed PCCD-A23
- net RTC-OE renamed ~{RTC-OE}
Changed lines of the file:
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@@
     )
   )
-  (global_label "27G-5" (shape input) (at 40.64 233.68 180) (fields_autoplaced)
+  (global_label "PCCD-A23" (shape input) (at 40.64 233.68 180) (fields_autoplaced)
     (effects (font (size 1.27 1.27)) (justify right))
     (property "Intersheet References" "${INTERSHEET_REFS}" (id 0) (at 0 0 0)
@@
     )
   )
-  (global_label "RTC-OE" (shape input) (at 227.33 247.65 180) (fields_autoplaced)
+  (global_label "~{RTC-OE}" (shape input) (at 227.33 247.65 180) (fields_autoplaced)
     (effects (font (size 1.27 1.27)) (justify right))
     (property "Intersheet References" "${INTERSHEET_REFS}" (id 0) (at 0 0 0)
@@
     )
   )
-  (global_label "27G-2" (shape input) (at 40.64 236.22 180) (fields_autoplaced)
+  (global_label "PCCD-A22" (shape input) (at 40.64 236.22 180) (fields_autoplaced)
     (effects (font (size 1.27 1.27)) (justify right))
     (property "Intersheet References" "${INTERSHEET_REFS}" (id 0) (at 0 0 0)

Commit message: Major board changes to give a rough render of the PCB
Parts:
- 29G1: footprint (none) -> Package_SO:SOIC-16_4.55x10.3mm_P1.27mm
