File: Schematics (KiCad)/GX700-PWB/JAMMA-IO.kicad_sch (KiCad schematic)
At the start: 57 parts, among them CN1 B10PSHF1A, CN17 B6P-VH, CN2 VGA-DSUB15, CN22 BS4PSHF1AA, CN3 B10PSHF1A, CN5 B12PSHF1A, CN6 BS4PSHF1AA, U2 ADC0834

Commit message: General Fixes
Connections:
- net 058232-4 renamed WDC-CC2
- net 058232-5 renamed WDC-CC1
- net EXT-OUT-LATCH renamed ~{EXT-OUT-CLK}
- net WD_KICK renamed WDC-CP
Changed lines of the file:
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@@
     )
   )
-  (global_label "EXT-OUT-LATCH" (shape input) (at 244.475 151.13 180) (fields_autoplaced)
+  (global_label "~{EXT-OUT-CLK}" (shape input) (at 244.475 151.13 180) (fields_autoplaced)
     (effects (font (size 1.27 1.27)) (justify right))
     (property "Intersheet References" "${INTERSHEET_REFS}" (id 0) (at 226.3665 151.0506 0)
@@
     )
   )
-  (global_label "058232-4" (shape input) (at 340.36 203.2 180) (fields_autoplaced)
+  (global_label "WDC-CC2" (shape input) (at 340.36 203.2 180) (fields_autoplaced)
     (effects (font (size 1.27 1.27)) (justify right))
     (property "Intersheet References" "${INTERSHEET_REFS}" (id 0) (at -10.16 111.76 0)
@@
     )
   )
-  (global_label "058232-5" (shape input) (at 340.36 200.66 180) (fields_autoplaced)
+  (global_label "WDC-CC1" (shape input) (at 340.36 200.66 180) (fields_autoplaced)
     (effects (font (size 1.27 1.27)) (justify right))
     (property "Intersheet References" "${INTERSHEET_REFS}" (id 0) (at -10.16 111.76 0)
@@
     )
   )
-  (global_label "WD_KICK" (shape input) (at 353.695 240.03 180) (fields_autoplaced)
+  (global_label "WDC-CP" (shape input) (at 353.695 240.03 180) (fields_autoplaced)
     (effects (font (size 1.27 1.27)) (justify right))
     (property "Intersheet References" "${INTERSHEET_REFS}" (id 0) (at 343.6298 239.9506 0)
@@
     )
   )
-  (global_label "WD_KICK" (shape input) (at 337.82 208.28 180) (fields_autoplaced)
+  (global_label "WDC-CP" (shape input) (at 337.82 208.28 180) (fields_autoplaced)
     (effects (font (size 1.27 1.27)) (justify right))
     (property "Intersheet References" "${INTERSHEET_REFS}" (id 0) (at -10.16 113.03 0)

Commit message: Major board changes to give a rough render of the PCB
Parts:
- renumbered 15B2 to 15B1, 15B1 to 24C1
Other:
- moved on the sheet: 058232/58460, 10B1, 12B1, 12B2, 14B1, 15B1, 20A1, 20C1, 24A1, 24C1, 24E1D, 24E1E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
