File: Schematics (KiCad)/GX700-PWB/Ksys573.kicad_sch (KiCad schematic)
At the start: 45 parts, among them CN10 TX15-80P-ST, CN21 TX15-30P-ST, U71 22J-X700A1 XC9536

Commit message: Added Symbols, PSX page
Added PSX CPU and GPU symbols, added a COH PSX skeleton schematic and also updated the JAMMA symbol and footprint as it was bad.
Parts:
- gave numbers to parts that had none: 1
Other:
- added sheet PSX-COH (PSX-COH.kicad_sch)

Commit message: General Fixes
Connections:
- net U71-4 is gone; now on net ~{FL-BANK-CP}: U71.4 (M4)
- net ~{EXP1} is gone; now on net ~{DMACK5}: 25T1.2 (Pin_2), 25T1.7 (Pin_7), CN10.a12 (Pin_a12), CN10.b14 (Pin_b14), U71.28 (M14)
- net ~{EXP2} is gone; now on net ~{EXP-CE}: CN10.a15 (Pin_a15), U71.36 (M9)
- net +5V: no longer C2.1, C3.1
- net DREQ5: no longer R287.1
- net VGA-CSYNC: now also R288.1; no longer R288.2
- net at 23L1.16 (B2), R289.2: now also R288.2; no longer R288.1
- net 22M-13 renamed IRQ10
- net IRQ10: no longer CN10.a16 (Pin_a16), CN10.b16 (Pin_b16)
- net 24E-13 renamed I2C-~{TX}/RX
- net 27G-12 renamed FBANK-A0
- net 27G-15 renamed FBANK-A1
- net 27G-2 renamed PCCD-A22
- net 27G-5 renamed PCCD-A23
- net 27G-6 renamed PCCD-A24
- net 27G-9 renamed PCCD-A25
- net EXP-B14 renamed ~{DMACK5}
- net EXT-OUT-LATCH renamed ~{EXT-OUT-CLK}
- net H8-TX-FLAG renamed H8-WR-CLK
- net RTC-OE renamed ~{RTC-OE}
- net U17-4 renamed ~{FL-BANK-CP}
- net U71-26 renamed ~{KCUS-CE}
- net U71-27 renamed ~{H8-RST-CLK}
- net U71-29 renamed ~{IDE-RST-CLK}
- net U71-34 renamed ~{IDE-CE}
- net U71-5 renamed ~{H8-CLR-RXF}
- net U71-6 renamed CART-FLAG-RST
- net WD_KICK renamed WDC-CP
- new net IRQ10-EXP: CN10.a16 (Pin_a16), CN10.b16 (Pin_b16)
Other:
- note added: "??"
- note added: "DMACK5 from PSX CPU"
- note added: "EXP-A Side"
- note added: "EXP-B Side"
- note added: "Expansion Port Select"
- note added: "Flash/PCCARD Device Select"
- note added: "H8 Write - Sets latch, H8 clears when data is read in"
- note added: "IO Test Header - DMA/IRQ Connections"
- note added: "PCMCIA Slots"
- note added: "Possible set up for PSX controllers/Lightugns"
- note added: "Sets "SDA" to TX or RX"
- note removed: "29G Low"
- note removed: "EXP-A*"
- note removed: "EXP-B*"
- note removed: "Expansion Port Select 1"
- note removed: "Expansion Port Select 2"
- note removed: "H8 16-bit data port"
- note removed: "IO Config Header - Not populated"
- note removed: "N/C?"
- note removed: "PCMCIA A22-A25"
- note removed: "Yes this header is joined like this. No, I do not know why."
- moved on the sheet: C2, C3, H1, H10, H11, H12, H13, H2, H3, H4, H5, H6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

Commit message: Restructuring
Connections:
- net U71-38 renamed CART-TX-FLAG
Other:
- note added: "1f000000"
- note added: "1f400000"
- note added: "1f480000"
- note added: "1f4C0000"
- note added: "1f500000"
- note added: "1f520000"
- note added: "1f540000"
- note added: "1f560000"
- note added: "1f5c0000"
- note added: "1f600000"
- note added: "1f620000"
- note added: "1f640000"
- note added: "1f680000 - Sets latch, H8 clears when data is read in"
- note added: "1f6a0000"
- note added: "1f700000 - Not connected to the socket, needs modding to use"
- note added: "1f??????"
- note added: "27G-19 OUT 8 ??"
- note added: "573 to Cart Data Present"
- note added: "Cart to 573 Data Present Reset"
- note added: "H8 Write"
- note added: "PCMCIA CE1"
- note added: "PSX-EXP Enable - Used to select PIO devices, so 573 enable"
- note removed: "27G-19 OUT 8"
- note removed: "35J-1 Reset A"
- note removed: "H8 Write - Sets latch, H8 clears when data is read in"
- note removed: "IDE-CS0 IDE-CS1"
- note removed: "PCMCIA CE1 - Not connected to the socket, needs modding to use"
- note removed: "PSX-EXP Enable - Used to select PIO devices, so 573 enable?"
- note removed: "Security Cart Pin 30?"
Changed lines of the file:
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@@
     (effects (font (size 1.27 1.27)) (justify left bottom))
   )
-  (text "IDE-CS0\nIDE-CS1" (at 214.63 205.105 180)
-    (effects (font (size 1.27 1.27)) (justify right bottom))
+  (text "1f640000" (at 325.12 222.885 0)
+    (effects (font (size 1.27 1.27)) (justify left bottom))
+  )
+  (text "1f680000 - Sets latch, H8 clears when data is read in"
+    (at 325.12 215.265 0)
+    (effects (font (size 1.27 1.27)) (justify left bottom))
+  )
+  (text "1f400000" (at 325.12 240.665 0)
+    (effects (font (size 1.27 1.27)) (justify left bottom))
   )
   (text "Direction —>" (at 364.49 111.125 0)
     (effects (font (size 1.27 1.27)) (justify left bottom))
   )
-  (text "H8 Write - Sets latch, H8 clears when data is read in"
-    (at 295.275 215.265 0)
+  (text "H8 Write" (at 295.275 215.265 0)
     (effects (font (size 1.27 1.27)) (justify left bottom))
   )
@@
   (text "IDE Bus CE" (at 295.275 227.965 0)
     (effects (font (size 1.27 1.27)) (justify left bottom))
+  )
+  (text "1f??????" (at 210.185 214.63 180)
+    (effects (font (size 1.27 1.27)) (justify right bottom))
   )
   (text "IO Test Header - DMA/IRQ Connections" (at 89.535 212.09 0)
@@
     (effects (font (size 1.27 1.27) italic) (justify left bottom))
   )
-  (text "PSX-EXP Enable - Used to select PIO devices, so 573 enable?"
+  (text "PSX-EXP Enable - Used to select PIO devices, so 573 enable"
     (at 295.275 210.185 0)
     (effects (font (size 1.27 1.27)) (justify left bottom))
@@
     (effects (font (size 1.27 1.27)) (justify left bottom))
   )
+  (text "1f700000 - Not connected to the socket, needs modding to use"
+    (at 325.12 230.505 0)
+    (effects (font (size 1.27 1.27)) (justify left bottom))
+  )
   (text "26E-11 H8 Reset toggle" (at 295.275 238.125 0)
     (effects (font (size 1.27 1.27)) (justify left bottom))
   )
+  (text "1f520000" (at 210.185 207.01 180)
+    (effects (font (size 1.27 1.27)) (justify right bottom))
+  )
   (text "PSX Data Bus to 573 Data Bus Level Shifters" (at 75.565 41.91 0)
     (effects (font (size 1.27 1.27)) (justify left bottom))
@@
     (effects (font (size 1.27 1.27)) (justify left bottom))
   )
+  (text "1f600000" (at 325.12 207.645 0)
+    (effects (font (size 1.27 1.27)) (justify left bottom))
+  )
+  (text "1f500000" (at 210.185 209.55 180)
+    (effects (font (size 1.27 1.27)) (justify right bottom))
+  )
   (text "RTC OE" (at 295.275 212.725 0)
     (effects (font (size 1.27 1.27)) (justify left bottom))
   )
-  (text "Security Cart Pin 30?" (at 295.275 217.805 0)
-    (effects (font (size 1.27 1.27)) (justify left bottom))
-  )
-  (text "21C-13 H8 Control Pin" (at 214.63 207.645 180)
+  (text "573 to Cart Data Present" (at 295.275 217.805 0)
+    (effects (font (size 1.27 1.27)) (justify left bottom))
+  )
+  (text "21C-13 H8 Control Pin" (at 194.31 207.645 180)
     (effects (font (size 1.27 1.27)) (justify right bottom))
   )
@@
     (effects (font (size 1.27 1.27)) (justify left bottom))
   )
+  (text "1f620000" (at 325.12 212.725 0)
+    (effects (font (size 1.27 1.27)) (justify left bottom))
+  )
   (text "EXP-A\nSide" (at 137.795 204.47 0)
     (effects (font (size 1.27 1.27)) (justify left bottom))
   )
-  (text "27G-19 OUT 8" (at 214.63 215.265 180)
+  (text "1f6a0000" (at 325.12 217.805 0)
+    (effects (font (size 1.27 1.27)) (justify left bottom))
+  )
+  (text "27G-19 OUT 8 ??" (at 194.31 214.63 180)
     (effects (font (size 1.27 1.27)) (justify right bottom))
   )
@@
     (effects (font (size 1.27 1.27)) (justify left bottom))
   )
+  (text "1f480000" (at 210.185 201.93 180)
+    (effects (font (size 1.27 1.27)) (justify right bottom))
+  )
   (text "Data bus 74245 chips enable" (at 295.275 225.425 0)
     (effects (font (size 1.27 1.27)) (justify left bottom))
   )
-  (text "27G CP\n" (at 207.01 210.185 0)
-    (effects (font (size 1.27 1.27)) (justify left bottom))
+  (text "1f5c0000" (at 325.12 205.105 0)
+    (effects (font (size 1.27 1.27)) (justify left bottom))
+  )
+  (text "27G CP\n" (at 194.31 210.185 180)
+    (effects (font (size 1.27 1.27)) (justify right bottom))
   )
   (text "IDE INT Request" (at 214.63 240.665 180)
@@
     (effects (font (size 1.27 1.27)) (justify left bottom))
   )
-  (text "PCMCIA CE1 - Not connected to the socket, needs modding to use"
-    (at 295.275 230.505 0)
+  (text "1f4C0000" (at 210.185 204.47 180)
+    (effects (font (size 1.27 1.27)) (justify right bottom))
+  )
+  (text "1f540000" (at 210.185 212.09 180)
+    (effects (font (size 1.27 1.27)) (justify right bottom))
+  )
+  (text "1f000000" (at 325.12 220.345 0)
+    (effects (font (size 1.27 1.27)) (justify left bottom))
+  )
+  (text "1f560000" (at 325.12 233.045 0)
+    (effects (font (size 1.27 1.27)) (justify left bottom))
+  )
+  (text "PCMCIA CE1 " (at 295.275 230.505 0)
     (effects (font (size 1.27 1.27)) (justify left bottom))
   )
@@
     (effects (font (size 1.27 1.27)) (justify left bottom))
   )
-  (text "35J-1 Reset A" (at 212.09 212.725 180)
+  (text "Cart to 573 Data Present Reset" (at 194.31 212.09 180)
     (effects (font (size 1.27 1.27)) (justify right bottom))
   )
@@
     )
   )
-  (global_label "U71-38" (shape output) (at 276.225 216.535 0) (fields_autoplaced)
-    (effects (font (size 1.27 1.27)) (justify left))
-    (property "Intersheet References" "${INTERSHEET_REFS}" (id 0) (at 286.2902 216.4556 0)
+  (global_label "CART-TX-FLAG" (shape output) (at 276.225 216.535 0) (fields_autoplaced)
+    (effects (font (size 1.27 1.27)) (justify left))
+    (property "Intersheet References" "${INTERSHEET_REFS}" (id 0) (at 292.9425 216.4556 0)
       (effects (font (size 1.27 1.27)) (justify left) hide)
     )

Commit message: Major board changes to give a rough render of the PCB
Parts:
- EXO-1: footprint Package_DIP:DIP-8_W10.16mm -> Package_DIP:DIP-8_W7.62mm
Connections:
- net +5V: no longer 30N1.16 (B2), 30N1.18 (B0), RA6.6 (R5), RA6.7 (R6)
- new net IO-ADDR-10: 30N1.16 (B2), RA6.7 (R6)
- new net IO-ADDR-8: 30N1.18 (B0), RA6.6 (R5)
Other:
- moved on the sheet: 27N1, 30N1, 32N1, C38, C39, RA4A
