File: Schematics (KiCad)/GX700-PWB/PSX-COH.kicad_sch (KiCad schematic)
At the start: 11 parts

Commit message: General Fixes
Parts:
- renumbered RA8 to RA12, RA9 to RA13, RA10 to RA14
Connections:
- net at RA12.1 (R1): now also CPU1.188 (GD23), GPU1.34 (GD23)
- net at RA12.2 (R2): now also CPU1.186 (GD21), GPU1.36 (GD21)
- net at RA12.3 (R3): now also CPU1.184 (GD19), GPU1.40 (GD19)
- net at RA12.4 (R4): now also CPU1.180 (GD17), GPU1.42 (GD17)
- net at R87.2: now also GPU1.4 (~{GPU-WR})
- net at RA13.1 (R1): now also CPU1.178 (GD15), GPU1.46 (GD15)
- net at RA13.2 (R2): now also CPU1.176 (GD13), GPU1.48 (GD13)
- net at RA13.3 (R3): now also CPU1.174 (GD11), GPU1.50 (GD11)
- net at RA13.4 (R4): now also CPU1.172 (GD9), GPU1.54 (GD9)
- net at RA14.1 (R1): now also CPU1.168 (GD7), GPU1.56 (GD7)
- net at RA14.2 (R2): now also CPU1.166 (GD5), GPU1.58 (GD5)
- net at RA14.3 (R3): now also CPU1.164 (GD3), GPU1.62 (GD3)
- net at RA14.4 (R4): now also CPU1.162 (GD1), GPU1.64 (GD1)
- net at GPU1.1 (~{GPU-CS}): now also R85.2
- net at GPU1.12 (~{DREQ}): now also CPU1.200 (GPU-DREQ)
- net at GPU1.13 (~{IRQ1}): now also CPU1.102 (~{INT1})
- net at GPU1.2 (GPU-A2): now also CPU1.153 (GA2)
- net at GPU1.206 (~{DSYSCLK}): now also R84.2
- net at GPU1.24 (GD31): now also CPU1.198 (GD31), RA11.1 (R1)
- net at GPU1.25 (GD30): now also CPU1.197 (GD30), RA11.9 (R8)
- net at GPU1.26 (GD29): now also CPU1.194 (GD29), RA11.2 (R2)
- net at GPU1.27 (GD28): now also CPU1.193 (GD28), RA11.8 (R7)
- net at GPU1.28 (GD27): now also CPU1.192 (GD27), RA11.3 (R3)
- net at GPU1.3 (~{GPU-RD}): now also R86.2
- net at GPU1.31 (GD26): now also CPU1.191 (GD26), RA11.7 (R6)
- net at GPU1.32 (GD25): now also CPU1.190 (GD25), RA11.4 (R4)
- net at GPU1.33 (GD24): now also CPU1.189 (GD24), RA11.6 (R5)
- net at GPU1.35 (GD22): now also CPU1.187 (GD22), RA12.9 (R8)
- net at GPU1.39 (GD20): now also CPU1.185 (GD20), RA12.8 (R7)
- net at GPU1.41 (GD18): now also CPU1.181 (GD18), RA12.7 (R6)
- net at GPU1.45 (GD16): now also CPU1.179 (GD16), RA12.6 (R5)
- net at GPU1.47 (GD14): now also CPU1.177 (GD14), RA13.9 (R8)
- net at GPU1.49 (GD12): now also CPU1.175 (GD12), RA13.8 (R7)
- net at GPU1.5 (~{DACK}): now also R83.2
- net at GPU1.53 (GD10): now also CPU1.173 (GD10), RA13.7 (R6)
- net at GPU1.55 (GD8): now also CPU1.169 (GD8), RA13.6 (R5)
- net at GPU1.57 (GD6): now also CPU1.167 (GD6), RA14.9 (R8)
- net at GPU1.59 (GD4): now also CPU1.165 (GD4), RA14.8 (R7)
- net at GPU1.6 (~{RESET}): now also CPU1.76 (~{RESET})
- net at GPU1.63 (GD2): now also CPU1.163 (GD2), RA14.7 (R6)
- net at GPU1.65 (GD0): now also CPU1.161 (GD0), RA14.6 (R5)
- net at GPU1.9 (~{SYS-CLK}): now also CPU1.201 (SYSCLK0)
Other:
- moved on the sheet: CPU1, GPU1, R83, R84, R85, R86, R87
