File: Schematics (KiCad)/GX700-PWB/Security-cart.kicad_sch (KiCad schematic)
At the start: 10 parts, among them CN4 SECURITY_CART

Commit message: Added Symbols, PSX page
Added PSX CPU and GPU symbols, added a COH PSX skeleton schematic and also updated the JAMMA symbol and footprint as it was bad.
Parts:
- gave numbers to parts that had none: 2
- renumbered 35J to 35J1
Changed lines of the file:
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@@
   (symbol (lib_id "74xx:74LS74") (at 217.17 123.19 0) (unit 2)
     (in_bom yes) (on_board yes)
-    (property "Reference" "35J" (id 0) (at 223.52 113.03 0))
+    (property "Reference" "35J1" (id 0) (at 223.52 113.03 0))
     (property "Value" "74LS74" (id 1) (at 223.52 115.57 0))
     (property "Footprint" "Package_SO:SO-14_3.9x8.65mm_P1.27mm" (id 2) (at 217.17 123.19 0)
@@
   (symbol (lib_id "74xx:74LS74") (at 217.17 96.52 0) (unit 1)
     (in_bom yes) (on_board yes)
-    (property "Reference" "35J" (id 0) (at 223.52 86.36 0))
+    (property "Reference" "35J1" (id 0) (at 223.52 86.36 0))
     (property "Value" "74LS74" (id 1) (at 223.52 88.9 0))
     (property "Footprint" "Package_SO:SO-14_3.9x8.65mm_P1.27mm" (id 2) (at 217.17 96.52 0)
@@
   (symbol (lib_id "power:+5V") (at 217.17 88.9 0) (unit 1)
     (in_bom yes) (on_board yes)
-    (property "Reference" "#PWR?" (id 0) (at 217.17 92.71 0)
+    (property "Reference" "#PWR0279" (id 0) (at 217.17 92.71 0)
       (effects (font (size 1.27 1.27)) hide)
     )
@@
   (symbol (lib_id "power:+5V") (at 217.17 115.57 0) (unit 1)
     (in_bom yes) (on_board yes)
-    (property "Reference" "#PWR?" (id 0) (at 217.17 119.38 0)
+    (property "Reference" "#PWR0278" (id 0) (at 217.17 119.38 0)
       (effects (font (size 1.27 1.27)) hide)
     )
@@
   (symbol (lib_id "power:+5V") (at 162.56 25.4 0) (unit 1)
     (in_bom yes) (on_board yes)
-    (property "Reference" "#PWR?" (id 0) (at 162.56 29.21 0)
+    (property "Reference" "#PWR0282" (id 0) (at 162.56 29.21 0)
       (effects (font (size 1.27 1.27)) hide)
     )
@@
   (symbol (lib_id "power:+5V") (at 137.16 25.4 0) (unit 1)
     (in_bom yes) (on_board yes)
-    (property "Reference" "#PWR?" (id 0) (at 137.16 29.21 0)
+    (property "Reference" "#PWR0281" (id 0) (at 137.16 29.21 0)
       (effects (font (size 1.27 1.27)) hide)
     )
@@
   (symbol (lib_id "74xx:74LS14") (at 222.25 71.12 0) (mirror y) (unit 6)
     (in_bom yes) (on_board yes)
-    (property "Reference" "24E?" (id 0) (at 238.76 67.31 0))
+    (property "Reference" "24E2" (id 0) (at 238.76 67.31 0))
     (property "Value" "74LS14" (id 1) (at 231.14 67.31 0))
     (property "Footprint" "Package_SO:SO-14_3.9x8.65mm_P1.27mm" (id 2) (at 222.25 71.12 0)
@@
   (symbol (lib_id "74xx:74LS125") (at 201.93 63.5 0) (mirror y) (unit 3)
     (in_bom yes) (on_board yes)
-    (property "Reference" "35H?" (id 0) (at 209.55 66.04 0))
+    (property "Reference" "35H2" (id 0) (at 209.55 66.04 0))
     (property "Value" "74LS125" (id 1) (at 210.82 68.58 0))
     (property "Footprint" "Package_SO:SO-14_3.9x8.65mm_P1.27mm" (id 2) (at 201.93 63.5 0)
@@
   (symbol (lib_id "power:GND") (at 139.7 71.12 90) (unit 1)
     (in_bom yes) (on_board yes)
-    (property "Reference" "#PWR?" (id 0) (at 146.05 71.12 0)
-      (effects (font (size 1.27 1.27)) hide)
-    )
+    (property "Reference" "#PWR0280" (id 0) (at 146.05 71.12 0)
+      (effects (font (size 1.27 1.27)) hide)
+    )

Commit message: General Fixes
Connections:
- net 24E-13 renamed I2C-~{TX}/RX
- net U17-6 renamed CART-FLAG-RST
Changed lines of the file:
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@@
     )
   )
-  (global_label "24E-13" (shape input) (at 233.68 71.12 0) (fields_autoplaced)
+  (global_label "I2C-~{TX}{slash}RX" (shape input) (at 233.68 71.12 0) (fields_autoplaced)
     (effects (font (size 1.27 1.27)) (justify left))
-    (property "Intersheet References" "${INTERSHEET_REFS}" (id 0) (at 0 0 0)
-      (effects (font (size 1.27 1.27)) hide)
+    (property "Intersheet References" "${INTERSHEET_REFS}" (id 0) (at 246.648 71.0406 0)
+      (effects (font (size 1.27 1.27)) (justify left) hide)
     )
   )
@@
     )
   )
-  (global_label "U17-6" (shape input) (at 214.63 106.68 180) (fields_autoplaced)
+  (global_label "CART-FLAG-RST" (shape input) (at 214.63 106.68 180) (fields_autoplaced)
     (effects (font (size 1.27 1.27)) (justify right))
-    (property "Intersheet References" "${INTERSHEET_REFS}" (id 0) (at 0 0 0)
-      (effects (font (size 1.27 1.27)) hide)
+    (property "Intersheet References" "${INTERSHEET_REFS}" (id 0) (at 196.6425 106.6006 0)
+      (effects (font (size 1.27 1.27)) (justify right) hide)
     )
   )

Commit message: Restructuring
Connections:
- net U71-38 renamed CART-TX-FLAG
- no-connect marks 2 -> 4
Other:
- note added: "573 to Cart Data Present"
- note added: "Cart to 573 Data Present"
Changed lines of the file:
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@@
   )
   (no_connect (at 123.19 86.36))
+  (no_connect (at 224.79 125.73))
+  (no_connect (at 224.79 99.06))
   (no_connect (at 135.89 86.36))
   (wire (pts (xy 66.04 133.35) (xy 66.04 134.62))
@@
     (effects (font (size 1.27 1.27)) (justify left bottom))
   )
+  (text "573 to Cart Data Present" (at 206.375 127 180)
+    (effects (font (size 1.27 1.27)) (justify right bottom))
+  )
   (text "In port" (at 167.64 106.68 0)
     (effects (font (size 1.27 1.27)) (justify left bottom))
@@
   (text "KCUS 98" (at 236.22 124.46 0)
     (effects (font (size 1.27 1.27)) (justify left bottom))
+  )
+  (text "Cart to 573 Data Present" (at 205.74 100.33 180)
+    (effects (font (size 1.27 1.27)) (justify right bottom))
   )
   (text "No connect?" (at 105.41 69.85 180)
@@
     )
   )
-  (global_label "35J-5" (shape input) (at 228.6 96.52 0) (fields_autoplaced)
-    (effects (font (size 1.27 1.27)) (justify left))
-    (property "Intersheet References" "${INTERSHEET_REFS}" (id 0) (at 0 0 0)
-      (effects (font (size 1.27 1.27)) hide)
+  (global_label "35J-5" (shape output) (at 228.6 96.52 0) (fields_autoplaced)
+    (effects (font (size 1.27 1.27)) (justify left))
+    (property "Intersheet References" "${INTERSHEET_REFS}" (id 0) (at 237.0928 96.4406 0)
+      (effects (font (size 1.27 1.27)) (justify left) hide)
     )
   )
@@
     )
   )
-  (global_label "CART-31" (shape input) (at 228.6 93.98 0) (fields_autoplaced)
-    (effects (font (size 1.27 1.27)) (justify left))
-    (property "Intersheet References" "${INTERSHEET_REFS}" (id 0) (at 0 0 0)
-      (effects (font (size 1.27 1.27)) hide)
+  (global_label "CART-31" (shape output) (at 228.6 93.98 0) (fields_autoplaced)
+    (effects (font (size 1.27 1.27)) (justify left))
+    (property "Intersheet References" "${INTERSHEET_REFS}" (id 0) (at 239.5118 93.9006 0)
+      (effects (font (size 1.27 1.27)) (justify left) hide)
     )
   )
@@
     )
   )
-  (global_label "U71-38" (shape input) (at 207.01 123.19 180) (fields_autoplaced)
-    (effects (font (size 1.27 1.27)) (justify right))
-    (property "Intersheet References" "${INTERSHEET_REFS}" (id 0) (at 0 0 0)
-      (effects (font (size 1.27 1.27)) hide)
+  (global_label "CART-TX-FLAG" (shape input) (at 207.01 123.19 180) (fields_autoplaced)
+    (effects (font (size 1.27 1.27)) (justify right))
+    (property "Intersheet References" "${INTERSHEET_REFS}" (id 0) (at 190.2925 123.1106 0)
+      (effects (font (size 1.27 1.27)) (justify right) hide)
     )
   )
@@
     )
   )
-  (global_label "CART-27" (shape input) (at 227.33 120.65 0) (fields_autoplaced)
-    (effects (font (size 1.27 1.27)) (justify left))
-    (property "Intersheet References" "${INTERSHEET_REFS}" (id 0) (at 0 0 0)
-      (effects (font (size 1.27 1.27)) hide)
+  (global_label "CART-27" (shape output) (at 227.33 120.65 0) (fields_autoplaced)
+    (effects (font (size 1.27 1.27)) (justify left))
+    (property "Intersheet References" "${INTERSHEET_REFS}" (id 0) (at 238.2418 120.5706 0)
+      (effects (font (size 1.27 1.27)) (justify left) hide)
     )
   )
@@
     )
   )
-  (global_label "35J-9" (shape input) (at 227.33 123.19 0) (fields_autoplaced)
-    (effects (font (size 1.27 1.27)) (justify left))
-    (property "Intersheet References" "${INTERSHEET_REFS}" (id 0) (at 0 0 0)
-      (effects (font (size 1.27 1.27)) hide)
-    )
-  )
+  (global_label "35J-9" (shape output) (at 227.33 123.19 0) (fields_autoplaced)
+    (effects (font (size 1.27 1.27)) (justify left))
+    (property "Intersheet References" "${INTERSHEET_REFS}" (id 0) (at 235.8228 123.1106 0)
+      (effects (font (size 1.27 1.27)) (justify left) hide)
+    )
+  )

Commit message: Major board changes to give a rough render of the PCB
Parts:
- renumbered 24E2 to 24E1, 35H2 to 35H1
Connections:
- no-connect marks 4 -> 6
