File: Extra Hardware/GN845-PWB(B)/Schematic/GN845-PWB.kicad_sch (KiCad schematic)
At the start: 117 parts

Commit message: Updated IO Boards and descriptions
Parts:
- 10E: value (none) -> XC9536PC44 / N845B1; footprint (none) -> Package_LCC:PLCC-44
- 10H, 10H? (x4): value (none) -> PC817; footprint (none) -> Package_DIP:DIP-4_W7.62mm
- 7B, 7D, 7F, 7H, 7J: value (none) -> 74HC14; footprint (none) -> Package_DIP:DIP-14_W7.62mm
- 7J: renamed from 7B?; value (none) -> 74HC14; footprint (none) -> Package_DIP:DIP-14_W7.62mm
- C1: value (none) -> 330uf 14v; footprint (none) -> Capacitor_THT:CP_Radial_D8.0mm_P3.50mm
- C11, C12, C13, C14, C15, C17, C4, C6, C7, C9: value (none) -> 100n; footprint (none) -> Capacitor_THT:C_Axial_L3.8mm_D2.6mm_P10.00mm_Horizontal
- C18, C19, C20, C21, C22, C25, C27, C28, C29, C30, C31, C32, C33, C34, C35, C36, C37, C38, C39, C40, C41, C42, C43, C44, C45, C50, C? (x9): value (none) -> EMI_Filter_LCL; footprint (none) -> Connector_PinSocket_2.54mm:PinSocket_1x03_P2.54mm_Vertical
- C23: value (none) -> 330uf 50v; footprint (none) -> Capacitor_THT:CP_Radial_D8.0mm_P3.50mm
- C24: value (none) -> 0.1uf 50v; footprint (none) -> Capacitor_THT:C_Disc_D4.7mm_W2.5mm_P5.00mm
- C3, C? (x2): value (none) -> 100n 25v; footprint (none) -> Capacitor_THT:C_Axial_L3.8mm_D2.6mm_P10.00mm_Horizontal
- CN1: value (none) -> B13PSHF1A; footprint (none) -> Connector_JST:JST_NH_B13P_SHD
- CN2, CN3, CN4, CN5, CN6: value (none) -> B11PSHF1A; footprint (none) -> Connector_JST:JST_NH_B11P_SHD
- CN7: value (none) -> B4P-VH; footprint (none) -> Connector_JST:JST_VH_B4P-VH-B_1x04_P3.96mm_Vertical
- D1: value (none) -> 10D1; footprint (none) -> Diode_THT:D_DO-41_SOD81_P10.16mm_Horizontal
- DA1: value (none) -> B1D9-1A; footprint (none) -> Package_SIP:SIP9_Housing
- DA2: value (none) -> B1D9-1C; footprint (none) -> Package_SIP:SIP9_Housing
- H? (x4): value (none) -> MountingHole_Pad; footprint (none) -> MountingHole:MountingHole_3.2mm_M3_DIN965_Pad
- JP? (x3): value (none) -> Jumper_NC_Small; footprint (none) -> Capacitor_THT:C_Rect_L7.0mm_W2.0mm_P5.00mm
- JP? (x7): value (none) -> Jumper_NO_Small; footprint (none) -> Capacitor_THT:C_Rect_L7.0mm_W2.0mm_P5.00mm
- JTAG: value (none) -> Conn_01x06
- R10, R13, R16, R19, R7: value (none) -> 1k; footprint (none) -> Resistor_THT:R_Axial_DIN0204_L3.6mm_D1.6mm_P5.08mm_Vertical
- R11, R14, R17, R20, R8: value (none) -> 10k; footprint (none) -> Resistor_THT:R_Axial_DIN0204_L3.6mm_D1.6mm_P5.08mm_Vertical
- R31, R32, R34, R35: value (none) -> 100; footprint (none) -> Resistor_THT:R_Axial_DIN0204_L3.6mm_D1.6mm_P5.08mm_Vertical
- RA1: value (none) -> 4.7k; footprint (none) -> Resistor_THT:R_Array_SIP9
- RA2: value (none) -> 330; footprint (none) -> Resistor_THT:R_Array_SIP9
- RA3, RA4, RA6, RA7, RA?: value (none) -> 1K; footprint (none) -> Resistor_THT:R_Array_SIP5
- TR1, TR2, TR3, TR4, TR5: value (none) -> 2SD2352; footprint (none) -> Package_TO_SOT_THT:TO-220-3_Horizontal_TabDown
- U?: value (none) -> L7805
Connections:
- net 7B-2: now also 10E.25 (M17)
- net 7D-2: now also 10E.24 (M17)
- net 7D-4: now also 10E.38 (M7); no longer 10E.39 (I/O/GSR)
- net 7F-10: now also 10E.3 (M2)
- net 7F-2: now also 10E.22 (M16)
- net 7F-4: now also 10E.44 (M2)
- net 7F-6: now also 10E.1 (M1)
- net 7F-8: now also 10E.2 (M1)
- net 7H-10: now also 10E.33 (M12)
- net 7H-4: now also 10E.4 (M4)
- net 7H-6: now also 10E.6 (I/O/GCK2)
- net 7H-8: now also 10E.7 (I/O/GCK3)
- net 7J-10: now also 10E.26 (M16)
- net 7J-2: now also 10E.39 (I/O/GSR)
- net 7J-4: now also 10E.29 (M13)
- net 7J-6: now also 10E.28 (M14)
- net 7J-8: now also 10E.27 (M15)
- net BT-C: now also 10E.8 (M6); no longer 10E.7 (I/O/GCK3)
- net J-DN: now also 10E.12 (M10); no longer 10E.11 (M9)
- net J-LF: now also 10E.11 (M9); no longer 10E.9 (M8)
- net J-RT: now also 10E.9 (M8); no longer 10E.8 (M6)
- net J-UP: now also 10E.13 (M11); no longer 10E.12 (M10)
- net at 10E.5 (I/O/GCK1): now also 7J.12
- no-connect marks 4 -> 10
Other:
- note added: "Also have seen a D2461"
- note added: "CCFL States"
- note added: "Center Sensors"
- note added: "Down Sensors"
- note added: "Error - Actually labelled 7L on the board"
- note added: "Left Sensors"
- note added: "Outputs ULDR + C Also Serial out on U and R"
- note added: "Right Sensors"
- note added: "Serial In Clock"
- note added: "Serial In Data"
- note added: "Up Sensors"
- moved on the sheet: 7JF

Commit message: Updated GN845(B)'s schematic
The schematic wrongly claimed there was a seperate LIGHT-GND. This is not true, it was ground, only the outer mounting holes and the LCL filters have a seperate ground (or can have one)
Connections:
- net 7B-2 is gone; now on net TR1-B: 10E.25 (M17)
- net 7D-2 is gone; now on net TR2-B: 10E.24 (M17)
- net 7F-2 is gone; now on net TR3-B: 10E.22 (M16)
- net 7H-2 is gone; now on net TR4-B: 10E.20 (M15)
- net 7J-2 is gone; now on net TR5-B: 10E.39 (I/O/GSR)
- net GND: now also C23.2, C?.3, C?.3, C?.3, C?.3, CN2.1 (Pin_1), CN2.11 (Pin_11), CN2.8 (Pin_8), CN3.1 (Pin_1), CN3.11 (Pin_11), CN3.8 (Pin_8), CN4.1 (Pin_1), CN4.11 (Pin_11), CN4.8 (Pin_8), CN5.1 (Pin_1), CN5.11 (Pin_11), CN5.8 (Pin_8), CN6.1 (Pin_1), CN6.11 (Pin_11), CN6.8 (Pin_8), R31.2, R32.2, R34.2, R34.2, TR1.3 (E), TR2.3 (E), TR3.3 (E), TR4.3 (E)
- net LIGHT-GND: no longer C23.2, C?.3, C?.3, C?.3, C?.3, CN2.1 (Pin_1), CN2.11 (Pin_11), CN2.8 (Pin_8), CN3.1 (Pin_1), CN3.11 (Pin_11), CN3.8 (Pin_8), CN4.1 (Pin_1), CN4.11 (Pin_11), CN4.8 (Pin_8), CN5.1 (Pin_1), CN5.11 (Pin_11), CN5.8 (Pin_8), CN6.1 (Pin_1), CN6.11 (Pin_11), CN6.8 (Pin_8), R31.2, R32.2, R34.2, R34.2, TR1.3 (E), TR2.3 (E), TR3.3 (E), TR4.3 (E)
Other:
- note added: "Would also be centre CCFL"
- note removed: "?"
- moved on the sheet: 10E, 7JF, C?, JTAG

Commit message: Started mapping out Digital IO board
Parts:
- added C10: 100n 25v, Capacitor_THT:C_Axial_L3.8mm_D2.6mm_P10.00mm_Horizontal, symbol Device:C_Small
- U1: renamed from U?; footprint (none) -> Package_TO_SOT_THT:TO-220-3_Horizontal_TabDown
- gave numbers to parts that had none: 30
- renumbered 10E to 10E1, 10H to 10H1, 7B to 7B1, 7D to 7D1, 7F to 7F1, 7H to 7H1, 7J to 7J1, C27 to C26, JTAG to JTAG1, R34 to R33
Connections:
- net +5V: now also C10.1
- net GND: now also C10.2; no longer C23.2, C52.3, C53.3, C54.3, C55.3
- net LIGHT-GND: now also C23.2, C52.3, C53.3, C54.3, C55.3
- net 12V-IN: now reaches C46.1, C47.1, C48.1, C49.1, CN7.1 (Pin_1), CN7.2 (Pin_2)
- net GND-IN: now reaches C52.1, C53.1, C54.1, C55.1, CN7.3 (Pin_3), CN7.4 (Pin_4)
