File: Extra Hardware/GX894-PWB(B)A/Schematic/GX894-PWB/GX894-PWB.kicad_sch (KiCad schematic)
At the start: 53 parts, among them CN11 B12PSHF1A, CN12 B13PSHF1A, CN13 B5PSHF1AA, CN14 B7PSHF1AA, CN15 B8PSHF1AA, CN16 B4PSHF1AA, CN17 B3PSHF1AA, CN18 B6PSHF1AA, CN2 TX-80, CN3 TX-80

Commit message: Started mapping out Digital IO board
Parts:
- removed CN2, CN3: TX-80, symbol Connector_Generic:Conn_02x40_Row_Letter_First
- removed U? (x20): PC847, Package_DIP:DIP-16_W7.62mm, symbol Isolator:PC847
- removed U?: ADM232A, symbol Interface_UART:ADM232A
- added 19A2: ADM232A, symbol Interface_UART:ADM232A
- added 26G2: 19.6608 MHz, Oscillator:Oscillator_SMD_SeikoEpson_SG8002JC-4Pin_10.5x5.0mm, symbol Oscillator:SG-8002JC
- added C11, C12, C2, C28, C29, C3, C6, C8: 0.1µf, Capacitor_SMD:C_0805_2012Metric, symbol Device:C_Small
- added C14, C15, C16, C17, C18, C19, C22, C23, C24, C25, C26, C27, C30, C31, C32, C33, C35, C36, C37, C38, C39, C40, C41, C42, C47, C48, C49, C50, C60, C61, C62, C63: 10nf, Capacitor_SMD:C_0805_2012Metric, symbol Device:C_Small
- added C20, C66, C81, C85: 1uf, Capacitor_SMD:C_0805_2012Metric, symbol Device:C_Small
- added C46: 0.01MC1K, Capacitor_THT:C_Disc_D4.7mm_W2.5mm_P5.00mm, symbol Device:Varistor
- added CN2, CN3: 573_EXP, Connectors:JAE-TX15-80P, symbol Konami:573_EXP
- added H1, H2, H3, H4, H5, H6, H7, H8: MountingHole, MountingHole:MountingHole_3.5mm, symbol Mechanical:MountingHole
- added R1, R13, R28: 100Ω, symbol Device:R_Small
- added R15, R18: 100, Resistor_THT:R_Axial_DIN0207_L6.3mm_D2.5mm_P10.16mm_Horizontal, symbol Device:R
- added R16, R17: 5.6k, Resistor_THT:R_Axial_DIN0207_L6.3mm_D2.5mm_P10.16mm_Horizontal, symbol Device:R
- added R20, RA2, RA3, RA4: 470Ω, Resistor_SMD:R_Array_Convex_5x1206, symbol Device:R_Network08
- added R25, R26, R27, R29: 220Ω, symbol Device:R_Small
- added RA1: 4.7Ω, Resistor_SMD:R_Array_Convex_5x1206, symbol Device:R_Network08
- added RA5: 2.2k, Resistor_SMD:R_Array_Convex_5x1206, symbol Device:R_Network08
- added U1, U100, U101, U102, U103, U11, U12, U16, U20, U25, U27, U32, U34, U35, U37, U39, U40, U41, U42, U43, U44, U45, U46, U47, U49, U50, U51, U53, U55, U56, U57, U60, U61, U63, U66, U71, U72, U73, U78, U82, U85, U89, U9, U90, U95, U96, U97, U98, U99: ZBF253D, Connector_PinSocket_2.54mm:PinSocket_1x02_P2.54mm_Vertical, symbol Device:FerriteBead_Small
- added U10, U13, U5, U7, U8: PC847, Package_DIP:DIP-16_W7.62mm, symbol Isolator:PC847
- added U6: HYC2485S, Package_SIP:SIP-8_19x3mm_P2.54mm, symbol Arcade_Network:HYC2485S
- 19D1: renamed from U?; footprint (none) -> Package_SO:SOIC-14_3.9x8.7mm_P1.27mm
- 26G1: renamed from X?; value SG-8002JC -> 29.45MHz
- 30C1: renamed from 30C; footprint Arcade:RCA -> Arcade:RCA_Mounting; symbol Connector:Conn_Coaxial -> Connector:Conn_Coaxial_Switched
- 30D1: renamed from 30D; footprint Arcade:RCA -> Arcade:RCA_Mounting; symbol Connector:Conn_Coaxial -> Connector:Conn_Coaxial_Switched
- gave numbers to parts that had none: 5
Connections:
- net +5V: now reaches 19D1.14 (VCC)
- net +5V: now also 19A1.16 (VCC), 19A2.16 (VCC), C20.1, C28.1, C3.1, C66.1, C81.1, C85.1, CN2.a1 (+5V), CN2.a2 (+5V), CN2.a3 (+5V), CN2.a4 (+5V), CN2.a5 (+5V), CN2.b1 (+5V), CN2.b2 (+5V), CN2.b3 (+5V), CN2.b4 (+5V), CN2.b5 (+5V), CN3.a1 (+5V), CN3.a2 (+5V), CN3.a3 (+5V), CN3.a4 (+5V), CN3.a5 (+5V), CN3.b1 (+5V), CN3.b2 (+5V), CN3.b3 (+5V), CN3.b4 (+5V), CN3.b5 (+5V), R20.10 (common), R20.5 (common), RA1.10 (common), RA1.5 (common), RA2.10 (common), RA2.5 (common), RA3.10 (common), RA3.5 (common), RA4.10 (common), RA4.5 (common), U46.1, U6.2 (VCC)
- net GND: now reaches 19D1.7 (GND)
- net GND: now also 19A1.15 (GND), 19D1.1, 19D1.3, 26G1.2 (GND), CN15.4 (Pin_4), CN17.3 (Pin_3), 19A2.10 (T2IN), 19A2.15 (GND), 19A2.8 (R2IN), 26G2.2 (GND), C11.1, C20.2, C30.2, C31.2, C32.2, C33.2, C46.2, C6.1, C66.2, C81.2, C85.2, CN2.a11 (GND), CN2.a13 (GND), CN2.a33 (GND), CN2.a34 (GND), CN2.a35 (GND), CN2.a8 (GND), CN2.a9 (GND), CN2.b11 (GND), CN2.b13 (GND), CN2.b33 (GND), CN2.b34 (GND), CN2.b35 (GND), CN2.b7 (GND), CN2.b9 (GND), CN3.a11 (GND), CN3.a13 (GND), CN3.a33 (GND), CN3.a34 (GND), CN3.a35 (GND), CN3.a8 (GND), CN3.a9 (GND), CN3.b11 (GND), CN3.b13 (GND), CN3.b33 (GND), CN3.b34 (GND), CN3.b35 (GND), CN3.b7 (GND), CN3.b9 (GND), R16.1, RA5.10 (common), RA5.5 (common), U12.1, U41.1, U47.1, U6.6 (GND)
- net at U3.13: now also U3.11, U3.15, U3.9, C18.2, C19.2, C38.2, C40.2, U50.1
- net at U3.14: now also C19.1, U98.1
- net at U3.3: now also RA3.2 (R2)
- net at CN13.1 (Pin_1): now also U45.2
- net at CN13.2 (Pin_2): now also U89.2
- net at CN13.3 (Pin_3): now also U71.2
- net at CN13.4 (Pin_4): now also U34.2
- net at CN13.5 (Pin_5): now also U40.2
- net at CN14.1 (Pin_1): now also U46.2
- net at CN14.2 (Pin_2): now also U20.2
- net at CN14.3 (Pin_3): now also U32.2
- net at CN14.4 (Pin_4): now also U49.2
- net at CN14.5 (Pin_5): now also U57.2
- net at CN14.6 (Pin_6): now also U12.2
- net at CN14.7 (Pin_7): now also U41.2
- net at U3.10: now also C38.1, U96.1
- net at U3.7: now also RA3.4 (R4)
- net at 30C1.1 (Pin): now also 30D1.1 (Pin), U6.5 (PH-A)
- net at 30C1.2 (Switch): now also R15.2
- net at 19D1.13: now also C30.1, R25.1
- net at U3.1: now also RA3.1 (R1)
- net at U3.16: now also C18.1, U99.1
- net at U4.1: now also RA3.9 (R8)
- net at U4.15: now also U4.11, U4.13, U4.9, C22.2, C23.2, C24.2, C25.2, U35.1
- net at U4.16: now also C22.1, U95.1
- net at C10.1 (Pin_1): now also U37.2
- net at C10.10 (Pin_10): now also U1.2
- net at C10.2 (Pin_2): now also U56.2
- net at C10.3 (Pin_3): now also U53.2
- net at C10.4 (Pin_4): now also U43.2
- net at C10.5 (Pin_5): now also U39.2
- net at C10.6 (Pin_6): now also U63.2
- net at C10.7 (Pin_7): now also U27.2
- net at C10.8 (Pin_8): now also U16.2
- net at C10.9 (Pin_9): now also U9.2
- net at U4.10: now also C25.1, U82.1
- net at U4.7: now also RA3.6 (R5)
- net at U4.12: now also C24.1, U90.1
- net at U4.5: now also RA3.7 (R6)
- net at U4.14: now also C23.1, U44.1
- net at U4.3: now also RA3.8 (R7)
- net at CN12.1 (Pin_1): now also U50.2
- net at CN12.10 (Pin_10): now also U82.2
- net at CN12.2 (Pin_2): now also U99.2
- net at CN12.3 (Pin_3): now also U98.2
- net at CN12.4 (Pin_4): now also U97.2
- net at CN12.5 (Pin_5): now also U96.2
- net at CN12.6 (Pin_6): now also U35.2
- net at CN12.7 (Pin_7): now also U95.2
- net at CN12.8 (Pin_8): now also U44.2
- net at CN12.9 (Pin_9): now also U90.2
- net FGPA-89: now reaches CN17.1 (Pin_1)
- net FGPA-89: now also 19A1.11 (T1IN)
- net FGPA-88: now reaches CN17.2 (Pin_2)
- net FGPA-88: now also 19A1.12 (R1OUT)
- net at 19D1.9: now also C33.1, R26.1
- net at CN15.1 (Pin_1): now also U11.2
- net at CN15.2 (Pin_2): now also U42.2
- net at CN15.3 (Pin_3): now also U47.2
- net at CN15.5 (Pin_5): now also U85.2
- net at CN15.6 (Pin_6): now also U78.2
- net at CN15.7 (Pin_7): now also U66.2
- net at CN15.8 (Pin_8): now also U55.2
- net at 19D1.5: now also C31.1, R29.1
- net at 19D1.11: now also C32.1, R27.1
- net at CN11.1 (Pin_1): now also U72.2
- net at CN11.10 (Pin_10): now also U100.2
- net at CN11.2 (Pin_2): now also U73.2
- net at CN11.3 (Pin_3): now also U61.2
- net at CN11.4 (Pin_4): now also U51.2
- net at CN11.5 (Pin_5): now also U103.2
- net at CN11.6 (Pin_6): now also U60.2
- net at CN11.7 (Pin_7): now also U25.2
- net at CN11.8 (Pin_8): now also U102.2
- net at CN11.9 (Pin_9): now also U101.2
- net at 19A1.1 (C1+): now also C8.2
- net FGPA-93: now reaches 19A1.10 (T2IN)
- net at 19A1.13 (R1IN): now also U42.1
- net at 19A1.14 (T1OUT): now also R28.1
- net at 19A1.2 (VS+): now also C28.2
- net at 19A1.3 (C1-): now also C8.1
- net at 19A1.4 (C2+): now also C29.2
- net at 19A1.5 (C2-): now also C29.1
- net at 19A1.6 (VS-): now also C11.2
- net at 19A1.7 (T2OUT): now also R13.1
- net at 19A1.8 (R2IN): now also U78.1
- net FGPA-90: now reaches 19A1.9 (R2OUT)
- net +3V3: now reaches 26G1.1 (OE)
- net +3V3: now also 26G1.4 (Vcc), 26G2.1 (OE), 26G2.4 (Vcc), CN2.a36 (+3V3), CN2.a37 (+3V3), CN2.a38 (+3V3), CN2.a39 (+3V3), CN2.a40 (+3V3), CN2.b36 (+3V3), CN2.b37 (+3V3), CN2.b38 (+3V3), CN2.b39 (+3V3), CN2.b40 (+3V3), CN3.a36 (+3V3), CN3.a37 (+3V3), CN3.a38 (+3V3), CN3.a39 (+3V3), CN3.a40 (+3V3), CN3.b36 (+3V3), CN3.b37 (+3V3), CN3.b38 (+3V3), CN3.b39 (+3V3), CN3.b40 (+3V3)
- net at U3.12: now also C40.1, U97.1
- net at U3.5: now also RA3.3 (R3)
- net at 30D1.2 (Switch): now also R18.1
- new net: C37.1, U10.16, U73.1
- new net: C48.1, U39.1, U7.10
- new net: C48.2, C49.2, C50.2, C60.2, U37.1, U7.11, U7.13, U7.15, U7.9
- new net: R27.2, RA1.3 (R3), RA5.3 (R3), U49.1
- new net: RA4.1 (R1), U5.1
- new net: C26.2, C27.2, C35.2, C36.2, U45.1, U5.11, U5.13, U5.15, U5.9
- new net: C26.1, U5.16, U89.1
- new net: C35.1, U34.1, U5.12
- new net: RA4.3 (R3), U5.5
- new net: C37.2, C61.2, C62.2, C63.2, U10.11, U10.13, U10.15, U10.9, U72.1
- new net: R28.2, U11.1
- new net: R13.2, U85.1
- new net: C49.1, U53.1, U7.14
- new net: C17.1, U100.1, U13.10
- new net: C62.1, U10.12, U51.1
- new net: C27.1, U5.14, U71.1
- new net: RA4.2 (R2), U5.3
- new net: C41.1, U8.12, U9.1
- new net: C39.2, C41.2, C42.2, C47.2, U63.1, U8.11, U8.13, U8.15, U8.9
- new net: C47.1, U27.1, U8.16
- new net: C42.1, U16.1, U8.14
- new net: R20.8 (R7), U8.3
- new net: R29.2, RA1.2 (R2), RA5.2 (R2), U32.1
- new net: C36.1, U40.1, U5.10
- new net: RA2.6 (R5), U13.7
- new net: C14.2, C15.2, C16.2, C17.2, U13.11, U13.13, U13.15, U13.9, U60.1
- new net: C63.1, U10.14, U61.1
- new net: 30C1.3 (Sheild), 30D1.3 (Sheild), C46.1, R15.1, R17.2, R18.2, U6.4 (PH-B)
- new net: RA2.1 (R1), U10.1
- new net: C50.1, U43.1, U7.12
- new net: R20.3 (R3), U7.5
- new net: R16.2, R17.1
- new net: R20.7 (R6), U8.5
- new net: RA2.3 (R3), U10.5
- new net: R20.1 (R1), U7.1
- new net: C60.1, U56.1, U7.16
- new net: R26.2, RA1.4 (R4), RA5.4 (R4), U57.1
- new net: C15.1, U102.1, U13.14
- new net: RA2.8 (R7), U13.3
- new net: R20.2 (R2), U7.3
- new net: RA2.2 (R2), U10.3
- new net: RA2.4 (R4), U10.7
- new net: RA2.7 (R6), U13.5
- new net: RA2.9 (R8), U13.1
- new net: R25.2, RA1.1 (R1), RA5.1 (R1), U20.1
- new net: RA4.4 (R4), U5.7
- new net: 19A2.1 (C1+), C2.2
- new net: 19A2.2 (VS+), C3.2
- new net: 19A2.3 (C1-), C2.1
- new net: 19A2.4 (C2+), C12.2
- new net: 19A2.5 (C2-), C12.1
- new net: 19A2.6 (VS-), C6.2
- new net: C39.1, U1.1, U8.10
- new net: R20.6 (R5), U8.7
- new net: C16.1, U101.1, U13.12
- new net: R20.9 (R8), U8.1
- new net: R20.4 (R4), U7.7
- new net: C14.1, U13.16, U25.1
- new net: C61.1, U10.10, U103.1
- new net: R1.2, U66.1
- new net 573-A0: CN2.a24 (A0), CN3.a24 (A0)
- new net 573-A1: CN2.b24 (A1), CN3.b24 (A1)
- new net 573-A12: CN2.a20 (A12), CN3.a20 (A12)
- new net 573-A13: CN2.b20 (A13), CN3.b20 (A13)
- new net 573-A14: CN2.a19 (A14), CN3.a19 (A14)
- new net 573-A15: CN2.b19 (A15), CN3.b19 (A15)
- new net 573-A2: CN2.a23 (A2), CN3.a23 (A2)
- new net 573-A20: CN2.a18 (A20), CN3.a18 (A20)
- new net 573-A21: CN2.b18 (A21), CN3.b18 (A21)
- new net 573-A22: CN2.a17 (A22), CN3.a17 (A22)
- new net 573-A23: CN2.b17 (A23), CN3.b17 (A23)
- new net 573-A3: CN2.b23 (A3), CN3.b23 (A3)
- new net 573-A4: CN2.a22 (A4), CN3.a22 (A4)
- new net 573-A5: CN2.b22 (A5), CN3.b22 (A5)
- new net 573-A6: CN2.a21 (A6), CN3.a21 (A6)
- new net 573-A7: CN2.b21 (A7), CN3.b21 (A7)
- new net 573-D0: CN2.a32 (D0), CN3.a32 (D0)
- new net 573-D1: CN2.b32 (D1), CN3.b32 (D1)
- new net 573-D10: CN2.a27 (D10), CN3.a27 (D10)
- new net 573-D11: CN2.b27 (D11), CN3.b27 (D11)
- new net 573-D12: CN2.a26 (D12), CN3.a26 (D12)
- new net 573-D13: CN2.b26 (D13), CN3.b26 (D13)
- new net 573-D14: CN2.a25 (D14), CN3.a25 (D14)
- new net 573-D15: CN2.b25 (D15), CN3.b25 (D15)
- new net 573-D2: CN2.a31 (D2), CN3.a31 (D2)
- new net 573-D3: CN2.b31 (D3), CN3.b31 (D3)
- new net 573-D4: CN2.a30 (D4), CN3.a30 (D4)
- new net 573-D5: CN2.b30 (D5), CN3.b30 (D5)
- new net 573-D6: CN2.a29 (D6), CN3.a29 (D6)
- new net 573-D7: CN2.b29 (D7), CN3.b29 (D7)
- new net 573-D8: CN2.a28 (D8), CN3.a28 (D8)
- new net 573-D9: CN2.b28 (D9), CN3.b28 (D9)
- new net DREQ5: CN2.a14 (DREQ5), CN3.a14 (DREQ5)
- new net DREQ5-2: CN2.b12 (DREQ5), CN3.b12 (DREQ5)
- new net EXP-15: CN2.b15 (N/C), CN3.b15 (N/C)
- new net FGPA-85: 19A2.12 (R1OUT)
- new net FGPA-87: 19A2.11 (T1IN)
- new net FPGA-100: U6.3 (~{TXEN})
- new net FPGA-98: U6.8 (RX)
- new net FPGA-99: U6.7 (TX)
- new net IRQ10: CN2.a16 (IRQ10), CN3.a16 (IRQ10)
- new net IRQ10-2: CN2.b16 (IRQ10), CN3.b16 (IRQ10)
- new net RX3: 19A2.13 (R1IN), U55.1
- new net TX3: 19A2.14 (T1OUT), R1.1
- new net ~{EXP1-2}: CN2.b14 (~{EXP1}), CN3.b14 (~{EXP1})
- new net ~{EXP1}: CN2.a12 (~{EXP1}), CN3.a12 (~{EXP1})
- new net ~{EXP2}: CN2.a15 (~{EXP2}), CN3.a15 (~{EXP2})
- new net ~{READ}: CN2.a6 (~{READ}), CN3.a6 (~{READ})
- new net ~{RESET2}: CN2.b10 (~{RESET}), CN3.b10 (~{RESET})
- new net ~{RESET}: CN2.a10 (~{RESET}), CN3.a10 (~{RESET})
- new net ~{WR1}: CN2.b6 (~{WR1}), CN3.b6 (~{WR1})
- new net ~{WR2}: CN2.a7 (~{WR2}), CN3.a7 (~{WR2})
- no-connect marks 0 -> 21
Other:
- note added: "ARCnet Physical Layer"
- note added: "Not populated (pass-thru?)"
- note added: "This document lists the transceiver as being ARCNET compatible. https://accelconf.web.cern.ch/icalepcs2013/papers/tuppc089.pdf"
- moved on the sheet: 19D1A, 19D1B, 19D1C, 19D1D, 19D1E, 19D1F, 19D1G, C10, CN11, CN12, CN13, CN14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
