File: Extra Hardware/Expansion Boards/GX894-PWB(B)A/Schematic/GX894-PWB/GX894-PWB.kicad_sch (KiCad schematic)
At the start: 147 parts, among them CN11 B12PSHF1A, CN12 B13PSHF1A, CN13 B5PSHF1AA, CN14 B7PSHF1AA, CN15 B8PSHF1AA, CN16 B4PSHF1AA, CN17 B3PSHF1AA, CN18 B6PSHF1AA, CN2 573_EXP, CN3 573_EXP, U1 ZBF253D, U10 PC847, U100 ZBF253D, U101 ZBF253D, U102 ZBF253D, U103 ZBF253D, U11 ZBF253D, U12 ZBF253D, U13 PC847, U16 ZBF253D, U2 XC9536PC44, U20 ZBF253D, U25 ZBF253D, U27 ZBF253D, U3 PC847, U32 ZBF253D, U34 ZBF253D, U35 ZBF253D, U37 ZBF253D, U39 ZBF253D, U4 PC847, U40 ZBF253D, U41 ZBF253D, U42 ZBF253D, U43 ZBF253D, U44 ZBF253D, U45 ZBF253D, U46 ZBF253D, U47 ZBF253D, U49 ZBF253D, U5 PC847, U50 ZBF253D, U51 ZBF253D, U53 ZBF253D, U55 ZBF253D, U56 ZBF253D, U57 ZBF253D, U6 HYC2485S, U60 ZBF253D, U61 ZBF253D, U63 ZBF253D, U66 ZBF253D, U7 PC847, U71 ZBF253D, U72 ZBF253D, U73 ZBF253D, U78 ZBF253D, U79 DS2401P, U8 PC847, U82 ZBF253D, U85 ZBF253D, U89 ZBF253D, U9 ZBF253D, U90 ZBF253D, U95 ZBF253D, U96 ZBF253D, U97 ZBF253D, U98 ZBF253D, U99 ZBF253D

Commit message: Major PCB changes to render a nicer 3D image
Connections:
- net RX3: no longer names the net of 19A2.13 (R1IN), U55.1
- net TX3: no longer names the net of 19A2.14 (T1OUT), R1.1
Other:
- note added: "CTS"
- note added: "DSR"
- note added: "DTR"
- note added: "GND"
- note added: "RTS"
- note added: "RX"
- note added: "TX"
- moved on the sheet: 19A1, 19A2, C11, C12, C2, C20, C28, C29, C3, C6, C8, CN15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
